File: aek.sch (KiCad schematic (older format))
At the start: 225 parts, among them J1 Conn_01x04_Shielded, SW1 SW_Push, U1 ATmega32U4-AU, Y1 16MHz

Commit message: updates
Parts:
- removed J1: Conn_01x04_Shielded, Connector_JST:JST_SH_BM04B-SRSS-TB_1x04-1MP_P1.00mm_Vertical, symbol Connector_Generic_Shielded:Conn_01x04_Shielded
- removed R1, R2: 22, Resistor_SMD:R_0805_2012Metric, symbol Device:R_Small
- added J1: Conn_01x04_MountingPin, Connector_JST:JST_SH_SM04B-SRSS-TB_1x04-1MP_P1.00mm_Horizontal, symbol Connector_Generic_MountingPin:Conn_01x04_MountingPin
- SW1: footprint MX_Alps_Hybrid:MX-1U-NoLED -> random-keyboard-parts:SKQG-1155865
Connections:
- wire segments 363 -> 359
Changed lines of the file:
@@
 Wire Wire Line
 	3700 4750 3400 4750
-$Comp
-L Connector_Generic_Shielded:Conn_01x04_Shielded J1
-U 1 1 6120F753
-P 3900 4850
-F 0 "J1" H 3988 4763 50  0000 L CNN
-F 1 "Conn_01x04_Shielded" H 3988 4672 50  0000 L CNN
-F 2 "Connector_JST:JST_SH_BM04B-SRSS-TB_1x04-1MP_P1.00mm_Vertical" H 3900 4850 50  0001 C CNN
-F 3 "~" H 3900 4850 50  0001 C CNN
-	1    3900 4850
-	1    0    0    -1
-$EndComp
 Connection ~ 3400 4500
 Wire Wire Line
@@
 	1    0    0    -1
 $EndComp
-Text GLabel 1150 5100 0    50   Input ~ 0
+Text GLabel 1950 5100 0    50   Input ~ 0
 D-
-Text GLabel 1150 5000 0    50   Input ~ 0
+Text GLabel 1950 5000 0    50   Input ~ 0
 D+
 $Comp
@@
 F 0 "SW1" H 1450 3705 50  0000 C CNN
 F 1 "SW_Push" H 1450 3614 50  0000 C CNN
-F 2 "MX_Alps_Hybrid:MX-1U-NoLED" H 1450 3450 60  0001 C CNN
+F 2 "random-keyboard-parts:SKQG-1155865" H 1450 3450 60  0001 C CNN
 F 3 "" H 1450 3450 60  0000 C CNN
 	1    1450 3450
@@
 $EndComp
 $Comp
-L Device:R_Small R1
-U 1 1 61202ECD
-P 1400 5100
-F 0 "R1" V 1204 5100 50  0000 C CNN
-F 1 "22" V 1295 5100 50  0000 C CNN
-F 2 "Resistor_SMD:R_0805_2012Metric" H 1400 5100 50  0001 C CNN
-F 3 "~" H 1400 5100 50  0001 C CNN
-	1    1400 5100
-	0    1    1    0
-$EndComp
-Wire Wire Line
-	1950 5100 1500 5100
-Wire Wire Line
-	1300 5100 1150 5100
-$Comp
-L Device:R_Small R2
-U 1 1 6120239A
-P 1550 5000
-F 0 "R2" V 1354 5000 50  0000 C CNN
-F 1 "22" V 1445 5000 50  0000 C CNN
-F 2 "Resistor_SMD:R_0805_2012Metric" H 1550 5000 50  0001 C CNN
-F 3 "~" H 1550 5000 50  0001 C CNN
-	1    1550 5000
-	0    1    1    0
-$EndComp
-Wire Wire Line
-	1650 5000 1950 5000
-Wire Wire Line
-	1450 5000 1150 5000
-$Comp
 L Device:C_Small C6
 U 1 1 6120621D
@@
 	1    0    0    -1
 $EndComp
+$Comp
+L Connector_Generic_MountingPin:Conn_01x04_MountingPin J1
+U 1 1 625405C4
+P 3900 4850
+F 0 "J1" H 3988 4764 50  0000 L CNN
+F 1 "Conn_01x04_MountingPin" H 3988 4673 50  0000 L CNN
+F 2 "Connector_JST:JST_SH_SM04B-SRSS-TB_1x04-1MP_P1.00mm_Horizontal" H 3900 4850 50  0001 C CNN
+F 3 "~" H 3900 4850 50  0001 C CNN
+	1    3900 4850
+	1    0    0    -1
+$EndComp

Commit message: updates
Parts:
- SW_CAP1: footprint MX_Alps_Hybrid:MX-2U-NoLED -> MX_Alps_Hybrid:MX-1.75U-NoLED
Changed lines of the file:
@@
 F 0 "SW_CAP1" H 6033 4023 60  0000 C CNN
 F 1 "MX-NoLED" H 6033 3949 20  0000 C CNN
-F 2 "MX_Alps_Hybrid:MX-2U-NoLED" H 5375 3775 60  0001 C CNN
+F 2 "MX_Alps_Hybrid:MX-1.75U-NoLED" H 5375 3775 60  0001 C CNN
 F 3 "" H 5375 3775 60  0001 C CNN
 	1    6000 3800
