File: aek.kicad_pcb (KiCad board)
At the start: 2 copper layers, 223 parts, among them J1 Conn_01x04_MountingPin, SW1 SW_Push, U1 ATmega32U4-AU, Y1 16MHz

Commit message: updates
Parts:
- D1, D10, D100, D101, D102, D103, D104, D109, D11, D110, D12, D13, D14, D15, D16, D17, D18, D19, D2, D20, D21, D22, D23, D24, D25, D26, D27, D28, D29, D3, D30, D31, D32, D33, D34, D35, D36, D37, D38, D39, D4, D40, D41, D42, D44, D45, D46, D47, D48, D49, D5, D50, D51, D52, D53, D54, D55, D56, D57, D58, D59, D6, D60, D61, D62, D63, D64, D65, D66, D67, D68, D69, D7, D70, D71, D72, D73, D74, D75, D76, D77, D78, D79, D8, D80, D81, D82, D83, D84, D85, D86, D87, D88, D89, D9, D90, D91, D92, D93, D94, D95, D96, D97, D98, D99: moved to B.Cu
- SW_CAP1: footprint MX_Alps_Hybrid:MX-2U-NoLED -> MX_Alps_Hybrid:MX-1.75U-NoLED
- moved D100 521.2 mm to (455.3, 33.3), turned to 90 degrees
- moved D1 514.7 mm to (38.1, 33.3), turned to 90 degrees
- moved D2 498.7 mm to (38.1, 71.4), turned to 90 degrees
- moved D12 485.2 mm to (76.2, 33.3), turned to 90 degrees
- moved D3 477.1 mm to (42.9, 90.5), turned to 90 degrees
- moved D101 475.7 mm to (436.2, 71.4), turned to 90 degrees
- moved D22 473.5 mm to (95.2, 33.3), turned to 90 degrees
- moved D11 473.1 mm to (57.1, 71.4), turned to 90 degrees
- moved D99 471.6 mm to (417.2, 71.4), turned to 90 degrees
- moved D13 467.5 mm to (76.2, 71.4), turned to 90 degrees
- moved D89 467.3 mm to (370.5, 33.3), turned to 90 degrees
- moved D88 458.4 mm to (351.5, 33.3), turned to 90 degrees
- moved D4 457.7 mm to (45.2, 109.5), turned to 90 degrees
- moved D102 456.8 mm to (436.2, 90.5), turned to 90 degrees
- moved D6 455.4 mm to (42.9, 147.6), turned to 90 degrees
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Routing:
- net D+: track 50.6 -> 0.77 mm
- net D-: track 49.2 -> 0.77 mm
- net +5V: track 85.7 -> 39.3 mm
- net GND: track 82.9 -> 41.0 mm
- net Net-(D20-Pad2): track 0.00 -> 8.89 mm
- net Net-(D10-Pad2): track 0.00 -> 8.21 mm
- net Net-(D40-Pad2): track 0.00 -> 8.21 mm

Commit message: updates
Parts:
- moved J1 87.0 mm to (483.8, 58.9)
- moved C3 59.4 mm to (430.0, 81.5)
- moved C7 59.4 mm to (441.6, 81.7)
- moved C2 59.4 mm to (422.1, 76.6)
- moved R3 59.4 mm to (445.9, 76.6)
- moved U1 59.4 mm to (434.0, 72.0)
- moved C1 59.4 mm to (429.1, 63.2)
- moved C4 59.4 mm to (438.7, 81.7)
- moved C5 59.4 mm to (424.5, 76.6)
- moved C6 59.4 mm to (443.5, 72.8)
- moved R4 59.4 mm to (424.5, 66.3)
- moved SW1 59.4 mm to (453.0, 74.1)
- moved Y1 59.4 mm to (434.5, 81.5)
- moved D76 55.1 mm to (331.3, 113.1)
- moved D83 55.1 mm to (406.6, 189.3)
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
Commit message: updates
Parts:
- moved D104 68.3 mm to (446.5, 129.9), turned to 0 degrees
- moved D100 67.1 mm to (446.5, 25.1), turned to 180 degrees
- moved D103 67.1 mm to (446.5, 101.3), turned to 0 degrees
- moved D109 67.1 mm to (446.5, 82.2), turned to 0 degrees
- moved D110 65.9 mm to (446.5, 64.8), turned to 0 degrees
- moved D85 53.6 mm to (398.9, 129.9)
- moved C2 53.6 mm to (386.8, 36.2)
- moved C3 53.6 mm to (394.7, 41.1)
- moved C7 53.6 mm to (406.3, 41.3)
- moved D76 53.6 mm to (296.0, 72.7)
- moved D87 53.6 mm to (371.3, 72.7)
- moved D90 53.6 mm to (398.9, 72.7)
- moved SW_INS1 53.6 mm to (323.7, 72.7)
- moved SW_KPASTR1 53.6 mm to (446.5, 72.7)
- moved D18 53.6 mm to (119.8, 129.9)
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
Commit message: base matrix
Routing:
- net ROW0: track 0.00 -> 544.9 mm
- net ROW10: track 0.00 -> 477.4 mm
- net Net-(D103-Pad1): track 0.00 -> 467.8 mm, vias 0 -> 4
- net ROW9: track 0.00 -> 463.9 mm, vias 0 -> 4
- net ROW4: track 0.00 -> 462.3 mm, vias 0 -> 4
- net ROW7: track 0.00 -> 448.7 mm, vias 0 -> 8
- net ROW8: track 0.00 -> 441.9 mm, vias 0 -> 8
- net ROW6: track 0.00 -> 434.5 mm, vias 0 -> 4
- net ROW5: track 0.00 -> 421.9 mm, vias 0 -> 2
- net ROW1: track 0.00 -> 403.9 mm
- net ROW2: track 0.00 -> 399.1 mm
- net COL6: track 0.00 -> 277.3 mm
- net COL5: track 0.00 -> 253.0 mm
- net COL2: track 0.00 -> 245.8 mm
- net COL7: track 0.00 -> 242.7 mm
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
Commit message: fix license
Parts:
- moved SW1 17.4 mm to (403.3, 43.5)
- moved C6 5.93 mm to (410.5, 26.9)
- moved R3 5.60 mm to (409.7, 41.8)
- moved C3 3.89 mm to (395.5, 37.3)
- moved C4 3.82 mm to (403.2, 37.5)
- moved R4 3.82 mm to (388.9, 22.1)
- moved C7 3.82 mm to (406.0, 37.5)
- moved Y1 3.82 mm to (398.9, 37.3)
- moved C1 3.82 mm to (393.5, 19.0)
- moved C5 3.82 mm to (388.9, 32.4)
- moved U1 3.82 mm to (398.4, 27.8)
- moved C2 3.82 mm to (386.5, 32.4)
Connections:
- net Net-(U1-Pad11) renamed ROW3
- U1 pad 10: Net-(U1-Pad10) -> ROW2
- U1 pad 12: Net-(U1-Pad12) -> ROW7
- U1 pad 18: Net-(U1-Pad18) -> ROW10
- U1 pad 19: Net-(U1-Pad19) -> COL0
- U1 pad 20: Net-(U1-Pad20) -> COL1
- U1 pad 21: Net-(U1-Pad21) -> COL2
- U1 pad 22: Net-(U1-Pad22) -> COL4
- U1 pad 25: Net-(U1-Pad25) -> COL3
- U1 pad 26: Net-(U1-Pad26) -> COL5
- U1 pad 27: Net-(U1-Pad27) -> COL6
- U1 pad 28: Net-(U1-Pad28) -> ROW4
- U1 pad 29: Net-(U1-Pad29) -> ROW5
- U1 pad 30: Net-(U1-Pad30) -> ROW6
- U1 pad 31: Net-(U1-Pad31) -> ROW8
- U1 pad 32: Net-(U1-Pad32) -> ROW9
- U1 pad 39: Net-(U1-Pad39) -> COL9
- U1 pad 40: Net-(U1-Pad40) -> COL8
- U1 pad 41: Net-(U1-Pad41) -> COL7
- U1 pad 8: Net-(U1-Pad8) -> ROW0
- U1 pad 9: Net-(U1-Pad9) -> ROW1
Routing:
- net ROW5: track 421.9 -> 536.5 mm, vias 2 -> 3
- net ROW0: track 544.9 -> 472.8 mm, vias 0 -> 1
- net ROW10: track 477.4 -> 420.0 mm, vias 0 -> 1
- net ROW8: track 441.9 -> 482.5 mm, vias 8 -> 10
- net ROW4: track 462.3 -> 499.8 mm, vias 4 -> 6
- net COL9: track 142.3 -> 172.8 mm
- net ROW1: track 403.9 -> 429.8 mm
- net ROW6: track 434.5 -> 459.5 mm, vias 4 -> 7
- net COL8: track 242.2 -> 255.6 mm, vias 0 -> 1
- net ROW2: track 399.1 -> 409.9 mm
- net GND: track 87.4 -> 79.6 mm, vias 4 -> 5
- net COL7: track 242.7 -> 246.3 mm, vias 0 -> 2
- net Net-(R3-Pad1): track 23.6 -> 20.2 mm, vias 2 -> 0
- net +5V: track 85.1 -> 88.3 mm
- net Net-(C6-Pad1): track 4.01 -> 6.77 mm
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Other:
- board outline added: 437.9 x 141 mm

Commit message: updates
Parts:
- added H2: MountingHole_Pad, MountingHole:MountingHole_2.7mm_M2.5_Pad, F.Cu at (24.8, 54.7)
- added H2: MountingHole_Pad, MountingHole:MountingHole_2.7mm_M2.5_Pad, F.Cu at (451.7, 54.7)
Routing:
- net GND: track 79.6 -> 154.7 mm, vias 5 -> 45
- net ROW7: track 448.7 -> 469.0 mm, vias 9 -> 10
- net ROW5: track 536.5 -> 527.5 mm
- net COL2: track 245.8 -> 253.5 mm
Other:
- outline, holes or cut-outs redrawn

Commit message: first draft
Parts:
- removed the H2 at (24.8, 54.7)
- added H1: MountingHole_Pad, MountingHole:MountingHole_2.7mm_M2.5_Pad, F.Cu at (24.8, 54.7)
- moved C3 1.95 mm to (396.0, 39.2)
- moved R3 1.23 mm to (408.9, 40.8)
- turned C1 to 180 degrees
Connections:
- D100 pad 1: ROW0 -> ROW10
- D103 pad 1: Net-(D103-Pad1) -> ROW3
- D109 pad 1: ROW9 -> ROW8
- D110 pad 1: ROW10 -> ROW9
- D15 pad 1: Net-(D103-Pad1) -> ROW3
- D26 pad 1: Net-(D103-Pad1) -> ROW3
- D37 pad 1: Net-(D103-Pad1) -> ROW3
- D4 pad 1: Net-(D103-Pad1) -> ROW3
- D48 pad 1: Net-(D103-Pad1) -> ROW3
- D59 pad 1: Net-(D103-Pad1) -> ROW3
- D70 pad 1: Net-(D103-Pad1) -> ROW3
- D81 pad 1: Net-(D103-Pad1) -> ROW3
- D92 pad 1: Net-(D103-Pad1) -> ROW3
- U1 pad 10: ROW2 -> ROW8
- U1 pad 18: ROW10 -> ROW4
- U1 pad 19: COL0 -> ROW6
- U1 pad 20: COL1 -> ROW5
- U1 pad 21: COL2 -> COL8
- U1 pad 22: COL4 -> ROW0
- U1 pad 25: COL3 -> COL7
- U1 pad 26: COL5 -> COL6
- U1 pad 27: COL6 -> COL5
- U1 pad 28: ROW4 -> COL4
- U1 pad 29: ROW5 -> COL3
- U1 pad 30: ROW6 -> COL2
- U1 pad 31: ROW8 -> COL1
- U1 pad 32: ROW9 -> COL0
- U1 pad 36: Net-(U1-Pad36) -> ROW9
- U1 pad 37: Net-(U1-Pad37) -> ROW1
- U1 pad 38: Net-(U1-Pad38) -> ROW10
- U1 pad 39: COL9 -> Net-(U1-Pad39)
- U1 pad 40: COL8 -> Net-(U1-Pad40)
- U1 pad 41: COL7 -> Net-(U1-Pad41)
- U1 pad 8: ROW0 -> COL9
- U1 pad 9: ROW1 -> ROW2
Routing:
- net ROW3: track 0.00 -> 591.1 mm, vias 0 -> 6
- net Net-(D103-Pad1): track 467.8 -> 0.00 mm, vias 4 -> 0
- net COL0: track 234.3 -> 617.7 mm, vias 0 -> 1
- net COL1: track 241.2 -> 565.2 mm, vias 0 -> 1
- net COL2: track 253.5 -> 539.0 mm, vias 0 -> 1
- net COL3: track 222.8 -> 460.1 mm, vias 0 -> 1
- net ROW6: track 459.5 -> 666.2 mm, vias 7 -> 8
- net COL4: track 237.6 -> 436.4 mm, vias 0 -> 1
- net ROW10: track 420.0 -> 594.6 mm, vias 1 -> 4
- net COL5: track 253.0 -> 403.5 mm, vias 0 -> 1
- net ROW8: track 482.5 -> 602.1 mm
- net COL6: track 277.3 -> 389.4 mm, vias 0 -> 1
- net ROW9: track 463.9 -> 572.1 mm, vias 4 -> 8
- net ROW7: track 469.0 -> 574.6 mm
- net ROW2: track 409.9 -> 491.3 mm, vias 0 -> 2
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
Commit message: clenaup
Routing:
- net ROW9: track 572.1 -> 559.0 mm
- net ROW1: track 491.4 -> 495.6 mm
- net ROW10: track 594.6 -> 593.0 mm, vias 4 -> 3
