File: aek.kicad_pcb (KiCad board)
At the start: 2 copper layers, 437.9 x 141 mm, 232 parts, among them J1 Conn_01x04_MountingPin, SW1 SW_Push, U1 ATmega32U4-AU, Y1 16MHz

Commit message: updates
Parts:
- moved C1 12.3 mm to (433.1, 35.3)
Routing:
- net +5V: track 147.6 -> 146.7 mm
Changed lines of the file:
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@@
     (thickness 1.6)
     (drawings 15)
-    (tracks 1677)
+    (tracks 1679)
     (zones 0)
     (modules 232)
@@
   )
   (module Capacitor_SMD:C_0805_2012Metric (layer B.Cu)
-    (at 420.93325 33.522 180)
+    (at 433.136 35.306 180)
     (descr "Capacitor SMD 0805 (2012 Metric), square (rectangular) end terminal, IPC_7351 nominal, (Body size source: IPC-SM-782 page 76, https://www.pcb-3d.com/wordpress/wp-content/uploads/ipc-sm-782a_amendment_1_and_2.pdf, https://docs.google.com/spreadsheets/d/1BsfQQcO9C6DZCsRaXUlFlo91Tg2WpOkGARC1WS5S8t0/edit?usp=sharing), generated with kicad-footprint-generator")
     (tags capacitor)
@@
   (segment (start 421.852 36.55325) (end 421.852 38.25325) (width 0.25) (layer B.Cu) (net 2) (status 10))
   (segment (start 421.88325 36.522) (end 421.852 36.55325) (width 0.25) (layer B.Cu) (net 2) (status 30))
-  (segment (start 421.88325 33.522) (end 421.88325 36.522) (width 0.25) (layer B.Cu) (net 2) (status 30))
   (segment (start 434.9005 52.8845) (end 436.372 54.356) (width 0.25) (layer B.Cu) (net 2) (status 20))
   (segment (start 433.477 52.8845) (end 434.9005 52.8845) (width 0.25) (layer B.Cu) (net 2) (status 10))
   (segment (start 432.87875 39.05325) (end 431.552 39.05325) (width 0.25) (layer B.Cu) (net 2) (status 20))
-  (segment (start 436.90325 35.02875) (end 432.87875 39.05325) (width 0.25) (layer B.Cu) (net 2))
   (segment (start 436.90325 29.17986) (end 436.90325 35.02875) (width 0.25) (layer B.Cu) (net 2))
   (segment (start 445.53236 20.55075) (end 436.90325 29.17986) (width 0.25) (layer B.Cu) (net 2))
@@
   (segment (start 430.470654 35.934596) (end 429.852 36.55325) (width 0.25) (layer B.Cu) (net 2))
   (segment (start 430.470654 35.120652) (end 430.470654 35.934596) (width 0.25) (layer B.Cu) (net 2))
+  (segment (start 434.086 36.322) (end 434.848 37.084) (width 0.25) (layer B.Cu) (net 2))
+  (segment (start 434.086 35.306) (end 434.086 36.322) (width 0.25) (layer B.Cu) (net 2))
+  (segment (start 434.848 37.084) (end 432.87875 39.05325) (width 0.25) (layer B.Cu) (net 2))
+  (segment (start 436.90325 35.02875) (end 434.848 37.084) (width 0.25) (layer B.Cu) (net 2))
   (segment (start 392.96581 29.616) (end 402.454 29.616) (width 0.25) (layer F.Cu) (net 142))
   (segment (start 392.07899 28.72918) (end 392.96581 29.616) (width 0.25) (layer F.Cu) (net 142))

Commit message: updates
Routing:
- net ROW1: track 493.2 -> 488.0 mm
- net GND: track 217.3 -> 213.2 mm
- net ROW10: track 581.3 -> 577.5 mm
- net ROW9: track 568.2 -> 564.6 mm
Changed lines of the file:
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@@
     (thickness 1.6)
     (drawings 15)
-    (tracks 1679)
+    (tracks 1666)
     (zones 0)
     (modules 232)
@@
   (segment (start 438.720678 52.582653) (end 438.800373 52.502958) (width 0.25) (layer F.Cu) (net 1))
   (segment (start 436.875347 52.582653) (end 438.720678 52.582653) (width 0.25) (layer F.Cu) (net 1))
-  (segment (start 418.47075 33.522) (end 416.327 35.66575) (width 0.25) (layer B.Cu) (net 1) (status 20))
-  (segment (start 419.98325 33.522) (end 418.47075 33.522) (width 0.25) (layer B.Cu) (net 1) (status 10))
-  (segment (start 421.03326 32.47199) (end 419.98325 33.522) (width 0.25) (layer B.Cu) (net 1) (status 20))
-  (segment (start 422.37143 32.47199) (end 421.03326 32.47199) (width 0.25) (layer B.Cu) (net 1))
-  (segment (start 422.70826 35.49699) (end 422.70826 32.80882) (width 0.25) (layer B.Cu) (net 1))
-  (segment (start 422.652 35.55325) (end 422.70826 35.49699) (width 0.25) (layer B.Cu) (net 1))
-  (segment (start 422.70826 32.80882) (end 422.37143 32.47199) (width 0.25) (layer B.Cu) (net 1))
-  (segment (start 422.652 36.55325) (end 422.652 35.55325) (width 0.25) (layer B.Cu) (net 1) (status 10))
   (segment (start 435.78825 40.31025) (end 434.64525 41.45325) (width 0.25) (layer B.Cu) (net 1))
   (segment (start 434.64525 41.45325) (end 431.552 41.45325) (width 0.25) (layer B.Cu) (net 1) (status 20))
@@
   (segment (start 429.052 34.844) (end 429.006 34.798) (width 0.25) (layer B.Cu) (net 1))
   (segment (start 429.052 36.55325) (end 429.052 34.844) (width 0.25) (layer B.Cu) (net 1))
+  (segment (start 416.514501 35.478249) (end 416.327 35.66575) (width 0.25) (layer B.Cu) (net 1))
+  (segment (start 422.576999 35.478249) (end 416.514501 35.478249) (width 0.25) (layer B.Cu) (net 1))
+  (segment (start 422.652 35.55325) (end 422.576999 35.478249) (width 0.25) (layer B.Cu) (net 1))
+  (segment (start 422.652 36.55325) (end 422.652 35.55325) (width 0.25) (layer B.Cu) (net 1))
   (segment (start 429.82075 36.5845) (end 429.852 36.55325) (width 0.25) (layer B.Cu) (net 2) (status 30))
   (segment (start 428.252 47.95325) (end 428.252 48.95325) (width 0.25) (layer B.Cu) (net 2) (status 10))
@@
   (segment (start 411.320989 52.991011) (end 411.320989 52.729991) (width 0.25) (layer B.Cu) (net 9))
   (segment (start 373.177499 75.132501) (end 377.495499 75.132501) (width 0.25) (layer B.Cu) (net 9))
-  (segment (start 424.252 33.07974) (end 422.744232 31.571972) (width 0.25) (layer B.Cu) (net 9))
-  (segment (start 424.252 36.55325) (end 424.252 33.07974) (width 0.25) (layer B.Cu) (net 9))
-  (segment (start 418.770029 31.571971) (end 418.258679 31.571971) (width 0.25) (layer B.Cu) (net 9))
   (segment (start 411.320989 45.242601) (end 411.320989 52.483011) (width 0.25) (layer B.Cu) (net 9))
   (segment (start 414.33199 42.2316) (end 411.320989 45.242601) (width 0.25) (layer B.Cu) (net 9))
@@
   (segment (start 414.274 35.55665) (end 414.274 38.354) (width 0.25) (layer B.Cu) (net 9))
   (segment (start 411.320989 52.483011) (end 411.320989 52.991011) (width 0.25) (layer B.Cu) (net 9))
-  (segment (start 418.25868 31.57197) (end 419.532028 31.57197) (width 0.25) (layer B.Cu) (net 9))
-  (segment (start 417.828325 32.002325) (end 418.25868 31.57197) (width 0.25) (layer B.Cu) (net 9))
-  (segment (start 422.744232 31.571972) (end 419.532029 31.571971) (width 0.25) (layer B.Cu) (net 9))
-  (segment (start 419.532028 31.57197) (end 419.532029 31.571971) (width 0.25) (layer B.Cu) (net 9))
-  (segment (start 419.532029 31.571971) (end 418.770029 31.571971) (width 0.25) (layer B.Cu) (net 9))
-  (segment (start 418.008029 31.822621) (end 417.828325 32.002325) (width 0.25) (layer B.Cu) (net 9))
-  (segment (start 417.828325 32.002325) (end 414.274 35.55665) (width 0.25) (layer B.Cu) (net 9))
   (segment (start 384.93559 59.31041) (end 385.064 59.182) (width 0.25) (layer F.Cu) (net 9))
   (segment (start 384.93559 60.706) (end 384.93559 59.31041) (width 0.25) (layer F.Cu) (net 9))
@@
   (segment (start 419.0365 82.2325) (end 376.4915 82.2325) (width 0.25) (layer B.Cu) (net 24))
   (segment (start 378.9045 82.2325) (end 376.4915 82.2325) (width 0.25) (layer B.Cu) (net 24))
-  (segment (start 410.870979 51.663021) (end 410.870979 53.492979) (width 0.25) (layer B.Cu) (net 24))
-  (segment (start 410.870979 45.056201) (end 410.870979 51.663021) (width 0.25) (layer B.Cu) (net 24))
-  (segment (start 413.766 42.16118) (end 410.870979 45.056201) (width 0.25) (layer B.Cu) (net 24))
-  (segment (start 413.766 35.42824) (end 413.766 42.16118) (width 0.25) (layer B.Cu) (net 24))
-  (segment (start 418.072279 31.121961) (end 413.766 35.42824) (width 0.25) (layer B.Cu) (net 24))
-  (segment (start 418.712037 31.121963) (end 418.712035 31.121961) (width 0.25) (layer B.Cu) (net 24))
-  (segment (start 422.930631 31.121963) (end 418.712037 31.121963) (width 0.25) (layer B.Cu) (net 24))
-  (segment (start 418.712035 31.121961) (end 418.072279 31.121961) (width 0.25) (layer B.Cu) (net 24))
-  (segment (start 425.052 33.243332) (end 422.930631 31.121963) (width 0.25) (layer B.Cu) (net 24))
-  (segment (start 425.052 36.55325) (end 425.052 33.243332) (width 0.25) (layer B.Cu) (net 24))
   (via (at 438.404 64.008) (size 0.8) (drill 0.4) (layers F.Cu B.Cu) (net 24))
   (segment (start 438.404 67.564) (end 440.27725 69.43725) (width 0.25) (layer F.Cu) (net 24))
@@
   (segment (start 55.062 68.2075) (end 57.912 71.0575) (width 0.25) (layer B.Cu) (net 25) (status 20))
   (segment (start 50.887 68.2075) (end 55.062 68.2075) (width 0.25) (layer B.Cu) (net 25) (status 10))
-  (segment (start 423.452 32.91615) (end 423.452 36.55325) (width 0.25) (layer B.Cu) (net 26) (status 20))
-  (segment (start 422.557831 32.021981) (end 423.452 32.91615) (width 0.25) (layer B.Cu) (net 26))
   (segment (start 57.912 74.3575) (end 62.483002 74.3575) (width 0.25) (layer B.Cu) (net 26) (status 10))
   (segment (start 96.012 36.2575) (end 97.7255 36.2575) (width 0.25) (layer B.Cu) (net 26) (status 10))
@@
   (segment (start 352.2345 44.1325) (end 352.2345 36.2575) (width 0.25) (layer B.Cu) (net 26) (status 20))
   (segment (start 411.770999 52.287001) (end 411.770999 52.795001) (width 0.25) (layer B.Cu) (net 26))
-  (segment (start 418.60998 32.02198) (end 418.44508 32.02198) (width 0.25) (layer B.Cu) (net 26))
-  (segment (start 418.44508 32.02198) (end 414.782 35.68506) (width 0.25) (layer B.Cu) (net 26))
-  (segment (start 418.60998 32.02198) (end 422.557831 32.021981) (width 0.25) (layer B.Cu) (net 26))
   (segment (start 414.782 42.418) (end 411.770999 45.429001) (width 0.25) (layer B.Cu) (net 26))
   (segment (start 414.782 35.68506) (end 414.782 42.418) (width 0.25) (layer B.Cu) (net 26))
@@
   (segment (start 434.848 37.084) (end 432.87875 39.05325) (width 0.25) (layer B.Cu) (net 2))
   (segment (start 436.90325 35.02875) (end 434.848 37.084) (width 0.25) (layer B.Cu) (net 2))
+  (segment (start 415.54713 34.28352) (end 415.288325 34.542325) (width 0.25) (layer B.Cu) (net 9))
+  (segment (start 424.252 35.55325) (end 422.98227 34.28352) (width 0.25) (layer B.Cu) (net 9))
+  (segment (start 422.98227 34.28352) (end 415.54713 34.28352) (width 0.25) (layer B.Cu) (net 9))
+  (segment (start 424.252 36.55325) (end 424.252 35.55325) (width 0.25) (layer B.Cu) (net 9))
+  (segment (start 415.288325 34.542325) (end 414.274 35.55665) (width 0.25) (layer B.Cu) (net 9))
+  (segment (start 425.052 35.55325) (end 425.052 36.55325) (width 0.25) (layer B.Cu) (net 24))
+  (segment (start 423.332261 33.833511) (end 425.052 35.55325) (width 0.25) (layer B.Cu) (net 24))
+  (segment (start 415.36073 33.83351) (end 423.332261 33.833511) (width 0.25) (layer B.Cu) (net 24))
+  (segment (start 413.766 42.16118) (end 413.766 35.42824) (width 0.25) (layer B.Cu) (net 24))
+  (segment (start 410.870979 45.056201) (end 413.766 42.16118) (width 0.25) (layer B.Cu) (net 24))
+  (segment (start 413.766 35.42824) (end 415.36073 33.83351) (width 0.25) (layer B.Cu) (net 24))
+  (segment (start 410.870979 53.492979) (end 410.870979 45.056201) (width 0.25) (layer B.Cu) (net 24))
+  (segment (start 423.452 35.55325) (end 423.452 36.55325) (width 0.25) (layer B.Cu) (net 26))
+  (segment (start 422.63228 34.73353) (end 423.452 35.55325) (width 0.25) (layer B.Cu) (net 26))
+  (segment (start 415.73353 34.73353) (end 422.63228 34.73353) (width 0.25) (layer B.Cu) (net 26))
+  (segment (start 415.73353 34.73353) (end 414.782 35.68506) (width 0.25) (layer B.Cu) (net 26))
   (segment (start 392.96581 29.616) (end 402.454 29.616) (width 0.25) (layer F.Cu) (net 142))
   (segment (start 392.07899 28.72918) (end 392.96581 29.616) (width 0.25) (layer F.Cu) (net 142))

Commit message: update
Connections:
- C10 pad 2: +5V -> Net-(C10-Pad2)
- C8 pad 2: +5V -> Net-(C10-Pad2)
- C9 pad 2: +5V -> Net-(C10-Pad2)
- LED1 pad 1: +5V -> Net-(C10-Pad2)
- LED2 pad 1: +5V -> Net-(C10-Pad2)
- LED3 pad 1: +5V -> Net-(C10-Pad2)
- U1 pad 18: ROW4 -> ROW1
- U1 pad 19: ROW6 -> ROW9
- U1 pad 20: ROW5 -> ROW10
- U1 pad 21: COL8 -> ROW4
- U1 pad 22: ROW0 -> ROW6
- U1 pad 25: COL7 -> ROW5
- U1 pad 26: COL6 -> COL8
- U1 pad 27: COL5 -> ROW0
- U1 pad 28: COL4 -> COL7
- U1 pad 29: COL3 -> COL6
- U1 pad 30: COL2 -> COL5
- U1 pad 31: COL1 -> COL4
- U1 pad 32: COL0 -> COL3
- U1 pad 36: ROW10 -> COL2
- U1 pad 37: ROW1 -> COL1
- U1 pad 38: ROW9 -> COL0
Routing:
- net ROW9: track 564.6 -> 538.5 mm, vias 7 -> 9
- net ROW10: track 577.5 -> 553.0 mm, vias 4 -> 5
- net ROW1: track 488.0 -> 468.1 mm
- net ROW5: track 561.5 -> 571.7 mm
- net COL8: track 327.0 -> 319.6 mm
- net ROW0: track 512.4 -> 506.3 mm
- net COL7: track 353.1 -> 347.0 mm
- net COL0: track 651.7 -> 656.8 mm
- net GND: track 213.2 -> 208.6 mm, vias 72 -> 70
- net ROW4: track 586.0 -> 583.6 mm
- net COL2: track 572.9 -> 574.9 mm
- net COL3: track 494.1 -> 492.6 mm
- net COL4: track 470.2 -> 468.8 mm
- net COL6: track 423.9 -> 422.7 mm
- net COL5: track 437.5 -> 436.5 mm
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
Commit message: updates
Parts:
- moved C1 1.27 mm to (433.1, 34.0)
Connections:
- C10 pad 2: Net-(C10-Pad2) -> +5V
- C8 pad 2: Net-(C10-Pad2) -> +5V
- C9 pad 2: Net-(C10-Pad2) -> +5V
- LED1 pad 1: Net-(C10-Pad2) -> +5V
- LED2 pad 1: Net-(C10-Pad2) -> +5V
- LED3 pad 1: Net-(C10-Pad2) -> +5V
Routing:
- net ROW6: track 677.3 -> 573.1 mm, vias 8 -> 6
- net ROW5: track 571.7 -> 575.7 mm, vias 3 -> 4
- net ROW2: track 509.7 -> 512.7 mm
- net ROW8: track 620.5 -> 622.9 mm
- net ROW9: track 538.5 -> 537.8 mm, vias 9 -> 8
- net +5V: track 146.7 -> 147.3 mm

Commit message: update
Routing:
- net GND: track 208.6 -> 206.0 mm
- net ROW6: track 573.1 -> 574.9 mm
Changed lines of the file:
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@@
     (thickness 1.6)
     (drawings 15)
-    (tracks 1627)
+    (tracks 1622)
     (zones 0)
     (modules 232)
@@
   (segment (start 427.4395 50.92825) (end 428.3895 50.92825) (width 0.25) (layer B.Cu) (net 1) (status 10))
   (via (at 135.382 153.162) (size 0.8) (drill 0.4) (layers F.Cu B.Cu) (net 1))
-  (via (at 135.128 146.304) (size 0.8) (drill 0.4) (layers F.Cu B.Cu) (net 1))
-  (segment (start 135.382 146.558) (end 135.128 146.304) (width 0.25) (layer F.Cu) (net 1))
+  (via (at 135.382 146.558) (size 0.8) (drill 0.4) (layers F.Cu B.Cu) (net 1))
   (segment (start 135.382 153.162) (end 135.382 146.558) (width 0.25) (layer F.Cu) (net 1))
   (via (at 93.218 116.84) (size 0.8) (drill 0.4) (layers F.Cu B.Cu) (net 1))
@@
   (segment (start 211.074 148.59) (end 213.36 148.59) (width 0.25) (layer F.Cu) (net 1))
   (via (at 317.246 136.652) (size 0.8) (drill 0.4) (layers F.Cu B.Cu) (net 1))
-  (via (at 316.992 130.556) (size 0.8) (drill 0.4) (layers F.Cu B.Cu) (net 1))
-  (segment (start 317.246 130.81) (end 316.992 130.556) (width 0.25) (layer F.Cu) (net 1))
+  (via (at 317.246 130.81) (size 0.8) (drill 0.4) (layers F.Cu B.Cu) (net 1))
   (segment (start 317.246 136.652) (end 317.246 130.81) (width 0.25) (layer F.Cu) (net 1))
   (via (at 270.002 62.484) (size 0.8) (drill 0.4) (layers F.Cu B.Cu) (net 1))
@@
   (segment (start 270.002 62.484) (end 270.002 66.802) (width 0.25) (layer F.Cu) (net 1))
   (via (at 308.864 104.394) (size 0.8) (drill 0.4) (layers F.Cu B.Cu) (net 1))
-  (via (at 308.356 99.06) (size 0.8) (drill 0.4) (layers F.Cu B.Cu) (net 1))
-  (segment (start 308.864 99.568) (end 308.356 99.06) (width 0.25) (layer F.Cu) (net 1))
+  (via (at 308.864 99.568) (size 0.8) (drill 0.4) (layers F.Cu B.Cu) (net 1))
   (segment (start 308.864 104.394) (end 308.864 99.568) (width 0.25) (layer F.Cu) (net 1))
   (via (at 276.098 72.898) (size 0.8) (drill 0.4) (layers F.Cu B.Cu) (net 1))
@@
   (via (at 355.092 73.914) (size 0.8) (drill 0.4) (layers F.Cu B.Cu) (net 1))
   (segment (start 355.092 76.454) (end 355.092 73.914) (width 0.25) (layer F.Cu) (net 1))
-  (via (at 361.442 135.128) (size 0.8) (drill 0.4) (layers F.Cu B.Cu) (net 1))
+  (via (at 362.204 135.128) (size 0.8) (drill 0.4) (layers F.Cu B.Cu) (net 1))
   (via (at 364.236 137.16) (size 0.8) (drill 0.4) (layers F.Cu B.Cu) (net 1))
   (segment (start 362.204 135.128) (end 364.236 137.16) (width 0.25) (layer F.Cu) (net 1))
-  (segment (start 361.442 135.128) (end 362.204 135.128) (width 0.25) (layer F.Cu) (net 1))
   (via (at 324.104 138.938) (size 0.8) (drill 0.4) (layers F.Cu B.Cu) (net 1))
   (via (at 327.152 136.906) (size 0.8) (drill 0.4) (layers F.Cu B.Cu) (net 1))
@@
   (segment (start 324.104 138.938) (end 325.12 138.938) (width 0.25) (layer F.Cu) (net 1))
   (via (at 259.588 135.128) (size 0.8) (drill 0.4) (layers F.Cu B.Cu) (net 1))
-  (via (at 259.842 132.08) (size 0.8) (drill 0.4) (layers F.Cu B.Cu) (net 1))
-  (segment (start 259.588 132.334) (end 259.842 132.08) (width 0.25) (layer F.Cu) (net 1))
+  (via (at 259.588 132.334) (size 0.8) (drill 0.4) (layers F.Cu B.Cu) (net 1))
   (segment (start 259.588 135.128) (end 259.588 132.334) (width 0.25) (layer F.Cu) (net 1))
   (via (at 206.502 102.87) (size 0.8) (drill 0.4) (layers F.Cu B.Cu) (net 1))
@@
   (via (at 187.96 114.554) (size 0.8) (drill 0.4) (layers F.Cu B.Cu) (net 18))
   (segment (start 182.118 120.396) (end 187.96 114.554) (width 0.25) (layer B.Cu) (net 18))
-  (via (at 188.214 111.76) (size 0.8) (drill 0.4) (layers F.Cu B.Cu) (net 18))
-  (segment (start 187.96 112.014) (end 188.214 111.76) (width 0.25) (layer F.Cu) (net 18))
-  (segment (start 187.96 114.554) (end 187.96 112.014) (width 0.25) (layer F.Cu) (net 18))
-  (segment (start 187.197 111.76) (end 186.4995 112.4575) (width 0.25) (layer B.Cu) (net 18) (status 20))
-  (segment (start 188.214 111.76) (end 187.197 111.76) (width 0.25) (layer B.Cu) (net 18))
+  (via (at 189.484 111.76) (size 0.8) (drill 0.4) (layers F.Cu B.Cu) (net 18))
   (segment (start 180.594 120.396) (end 228.346 120.396) (width 0.25) (layer B.Cu) (net 18))
   (segment (start 167.371002 120.396) (end 180.594 120.396) (width 0.25) (layer B.Cu) (net 18))
@@
   (segment (start 413.541796 59.82248) (end 413.541796 56.263454) (width 0.25) (layer B.Cu) (net 18))
   (segment (start 413.299387 60.064889) (end 413.541796 59.82248) (width 0.25) (layer B.Cu) (net 18))
+  (segment (start 188.7865 112.4575) (end 189.484 111.76) (width 0.25) (layer B.Cu) (net 18))
+  (segment (start 186.4995 112.4575) (end 188.7865 112.4575) (width 0.25) (layer B.Cu) (net 18))
+  (segment (start 189.484 113.03) (end 187.96 114.554) (width 0.25) (layer F.Cu) (net 18))
+  (segment (start 189.484 111.76) (end 189.484 113.03) (width 0.25) (layer F.Cu) (net 18))
   (segment (start 78.8745 125.3575) (end 81.7245 128.2075) (width 0.25) (layer B.Cu) (net 19) (status 20))
   (segment (start 74.6995 125.3575) (end 78.8745 125.3575) (width 0.25) (layer B.Cu) (net 19) (status 10))

Commit message: updates
Routing:
- net ROW1: track 467.7 -> 436.6 mm, vias 4 -> 2
- net COL3: track 492.6 -> 470.5 mm
- net COL2: track 574.9 -> 577.0 mm
- net COL1: track 602.7 -> 604.8 mm
- net COL0: track 656.8 -> 658.7 mm
- net ROW5: track 575.7 -> 574.9 mm

Commit message: updates
Other:
- board size 437.9 x 141 mm -> 437.9 x 142.7 mm
Changed lines of the file:
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@@
   (gr_circle (center 166.304 52.73) (end 172.304 52.73) (layer Edge.Cuts) (width 0.05))
   (gr_circle (center 310.204 52.73) (end 316.204 52.73) (layer Edge.Cuts) (width 0.05))
-  (gr_line (start 19.304 17.78) (end 19.304 152.654) (layer Edge.Cuts) (width 0.05))
-  (gr_line (start 457.2 152.654) (end 457.2 17.78) (layer Edge.Cuts) (width 0.05))
-  (gr_line (start 22.352 155.702) (end 454.152 155.702) (layer Edge.Cuts) (width 0.05))
-  (gr_arc (start 22.352 152.654) (end 19.304 152.654) (angle -90) (layer Edge.Cuts) (width 0.15))
+  (gr_line (start 19.304 17.78) (end 19.304 154.432) (layer Edge.Cuts) (width 0.05))
+  (gr_line (start 457.2 154.432) (end 457.2 17.78) (layer Edge.Cuts) (width 0.05))
+  (gr_line (start 22.352 157.462) (end 454.152 157.462) (layer Edge.Cuts) (width 0.05))
+  (gr_arc (start 22.352 154.432) (end 19.304 154.432) (angle -90) (layer Edge.Cuts) (width 0.15))
   (gr_arc (start 22.352 17.78) (end 22.352 14.732) (angle -90) (layer Edge.Cuts) (width 0.15))
-  (gr_arc (start 454.152 152.654) (end 454.152 155.702) (angle -90) (layer Edge.Cuts) (width 0.15))
+  (gr_arc (start 454.152 154.432) (end 454.152 157.48) (angle -90) (layer Edge.Cuts) (width 0.15))
   (gr_arc (start 454.152 17.78) (end 457.2 17.78) (angle -90) (layer Edge.Cuts) (width 0.15))
   (via (at 429.006 52.324) (size 0.8) (drill 0.4) (layers F.Cu B.Cu) (net 1))
@@
     (polygon
       (pts
-        (xy 458.216 156.464) (xy 18.796 156.21) (xy 18.542 13.97) (xy 457.962 14.224)
+        (xy 457.962 159.258) (xy 18.796 159.258) (xy 18.796 13.97) (xy 457.962 13.97)
       )
     )

Commit message: tweaks
Routing:
- net GND: track 206.0 -> 205.1 mm
