File: aek.kicad_sch (KiCad schematic)
At the start: 239 parts, among them J1 Conn_01x04_MountingPin, SW1 SW_Push, U1 ATmega32U4-AU, Y1 16MHz

Commit message: fix schematic issue
Parts:
- SW_KP0ALT1, SW_KPENTERALT1, SW_KPENTERX1: footprint MX_Alps_Hybrid:MX-2U-ReversedStabilizers-NoLED -> MX_Alps_Hybrid:MX-1U-NoLED
- gave numbers to parts that had none: 2
Connections:
- net ROW6: no longer D84.2 (A), SW_KP0.2 (ROW), SW_KP0ALT1.2 (ROW)
- new net: D84.2 (A), SW_KP0.2 (ROW), SW_KP0ALT1.2 (ROW)
Changed lines of the file:
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@@
   (junction (at 297.18 132.08) (diameter 1.016) (color 0 0 0 0))
   (junction (at 297.18 151.13) (diameter 1.016) (color 0 0 0 0))
-  (junction (at 297.18 170.18) (diameter 1.016) (color 0 0 0 0))
   (junction (at 297.18 189.23) (diameter 1.016) (color 0 0 0 0))
   (junction (at 297.18 208.28) (diameter 1.016) (color 0 0 0 0))
@@
   (junction (at 304.8 198.12) (diameter 1.016) (color 0 0 0 0))
   (junction (at 304.8 217.17) (diameter 1.016) (color 0 0 0 0))
-  (junction (at 314.96 165.1) (diameter 1.016) (color 0 0 0 0))
   (junction (at 317.5 127) (diameter 1.016) (color 0 0 0 0))
   (junction (at 322.58 64.77) (diameter 1.016) (color 0 0 0 0))
@@
     (stroke (width 0) (type solid) (color 0 0 0 0))
   )
-  (wire (pts (xy 281.94 165.1) (xy 293.37 165.1))
-    (stroke (width 0) (type solid) (color 0 0 0 0))
-  )
   (wire (pts (xy 287.02 45.72) (xy 287.02 36.83))
     (stroke (width 0) (type solid) (color 0 0 0 0))
@@
     (stroke (width 0) (type solid) (color 0 0 0 0))
   )
-  (wire (pts (xy 293.37 162.56) (xy 311.15 162.56))
+  (wire (pts (xy 289.56 161.29) (xy 289.56 165.1))
     (stroke (width 0) (type solid) (color 0 0 0 0))
   )
-  (wire (pts (xy 293.37 165.1) (xy 293.37 162.56))
+  (wire (pts (xy 289.56 165.1) (xy 281.94 165.1))
     (stroke (width 0) (type solid) (color 0 0 0 0))
   )
@@
     (stroke (width 0) (type solid) (color 0 0 0 0))
   )
-  (wire (pts (xy 297.18 170.18) (xy 314.96 170.18))
-    (stroke (width 0) (type solid) (color 0 0 0 0))
-  )
   (wire (pts (xy 297.18 184.15) (xy 299.72 184.15))
     (stroke (width 0) (type solid) (color 0 0 0 0))
@@
     (stroke (width 0) (type solid) (color 0 0 0 0))
   )
-  (wire (pts (xy 311.15 162.56) (xy 311.15 165.1))
+  (wire (pts (xy 311.15 161.29) (xy 289.56 161.29))
     (stroke (width 0) (type solid) (color 0 0 0 0))
   )
-  (wire (pts (xy 311.15 165.1) (xy 314.96 165.1))
+  (wire (pts (xy 311.15 165.1) (xy 311.15 161.29))
     (stroke (width 0) (type solid) (color 0 0 0 0))
   )
@@
     (stroke (width 0) (type solid) (color 0 0 0 0))
   )
-  (wire (pts (xy 314.96 165.1) (xy 314.96 170.18))
+  (wire (pts (xy 314.96 165.1) (xy 311.15 165.1))
     (stroke (width 0) (type solid) (color 0 0 0 0))
   )
@@
   (symbol (lib_id "Device:D_Small") (at 314.96 186.69 90) (unit 1)
     (in_bom yes) (on_board yes)
-    (property "Reference" "D?" (id 0) (at 316.738 185.5216 90)
+    (property "Reference" "D43" (id 0) (at 316.738 185.5216 90)
       (effects (font (size 1.27 1.27)) (justify right))
     )
@@
   (symbol (lib_id "Device:D_Small") (at 317.5 148.59 90) (unit 1)
     (in_bom yes) (on_board yes)
-    (property "Reference" "D?" (id 0) (at 319.278 147.4216 90)
+    (property "Reference" "D105" (id 0) (at 319.278 147.4216 90)
       (effects (font (size 1.27 1.27)) (justify right))
     )
@@
       (effects (font (size 0.508 0.508)))
     )
-    (property "Footprint" "MX_Alps_Hybrid:MX-2U-ReversedStabilizers-NoLED" (id 2) (at 300.355 161.925 0)
+    (property "Footprint" "MX_Alps_Hybrid:MX-1U-NoLED" (id 2) (at 300.355 161.925 0)
       (effects (font (size 1.524 1.524)) hide)
     )
@@
       (effects (font (size 0.508 0.508)))
     )
-    (property "Footprint" "MX_Alps_Hybrid:MX-2U-ReversedStabilizers-NoLED" (id 2) (at 302.895 142.875 0)
+    (property "Footprint" "MX_Alps_Hybrid:MX-1U-NoLED" (id 2) (at 302.895 142.875 0)
       (effects (font (size 1.524 1.524)) hide)
     )
@@
       (effects (font (size 0.508 0.508)))
     )
-    (property "Footprint" "MX_Alps_Hybrid:MX-2U-ReversedStabilizers-NoLED" (id 2) (at 323.215 123.825 0)
+    (property "Footprint" "MX_Alps_Hybrid:MX-1U-NoLED" (id 2) (at 323.215 123.825 0)
       (effects (font (size 1.524 1.524)) hide)
     )
@@
       (reference "D42") (unit 1) (value "D_Small") (footprint "Diode_SMD:D_SOD-123")
     )
+    (path "/0a9f023d-4fb2-47e0-ae5e-92c3e1654ff1"
+      (reference "D43") (unit 1) (value "D_Small") (footprint "Diode_SMD:D_SOD-123")
+    )
     (path "/00000000-0000-0000-0000-00006145a3a3"
       (reference "D44") (unit 1) (value "D_Small") (footprint "Diode_SMD:D_SOD-123")
@@
       (reference "D104") (unit 1) (value "D_Small") (footprint "Diode_SMD:D_SOD-123")
     )
+    (path "/d2e42852-7fb4-474f-a864-b3c20a8b77a0"
+      (reference "D105") (unit 1) (value "D_Small") (footprint "Diode_SMD:D_SOD-123")
+    )
     (path "/00000000-0000-0000-0000-00006145a285"
       (reference "D109") (unit 1) (value "D_Small") (footprint "Diode_SMD:D_SOD-123")
@@
       (reference "D110") (unit 1) (value "D_Small") (footprint "Diode_SMD:D_SOD-123")
     )
-    (path "/0a9f023d-4fb2-47e0-ae5e-92c3e1654ff1"
-      (reference "D?") (unit 1) (value "D_Small") (footprint "Diode_SMD:D_SOD-123")
-    )
-    (path "/d2e42852-7fb4-474f-a864-b3c20a8b77a0"
-      (reference "D?") (unit 1) (value "D_Small") (footprint "Diode_SMD:D_SOD-123")
-    )
     (path "/00000000-0000-0000-0000-000061db0c88"
       (reference "H1") (unit 1) (value "MountingHole_Pad") (footprint "MountingHole:MountingHole_2.7mm_M2.5_Pad")
@@
     )
     (path "/764d3922-6c3b-4ad1-99f1-13051e884ac2"
-      (reference "SW_KP0ALT1") (unit 1) (value "MX-NoLED") (footprint "MX_Alps_Hybrid:MX-2U-ReversedStabilizers-NoLED")
+      (reference "SW_KP0ALT1") (unit 1) (value "MX-NoLED") (footprint "MX_Alps_Hybrid:MX-1U-NoLED")
     )
     (path "/204e0ee4-dec0-4dc2-b622-9ea13958f955"
@@
     )
     (path "/4f0dc72b-fb67-4861-96c0-74fd1311c468"
-      (reference "SW_KPENTERALT1") (unit 1) (value "MX-NoLED") (footprint "MX_Alps_Hybrid:MX-2U-ReversedStabilizers-NoLED")
+      (reference "SW_KPENTERALT1") (unit 1) (value "MX-NoLED") (footprint "MX_Alps_Hybrid:MX-1U-NoLED")
     )
     (path "/045dc86d-b269-41b1-9424-1a177a9b131f"
-      (reference "SW_KPENTERX1") (unit 1) (value "MX-NoLED") (footprint "MX_Alps_Hybrid:MX-2U-ReversedStabilizers-NoLED")
+      (reference "SW_KPENTERX1") (unit 1) (value "MX-NoLED") (footprint "MX_Alps_Hybrid:MX-1U-NoLED")
     )
     (path "/00000000-0000-0000-0000-00006145a32b"

Commit message: updates
Parts:
- added R2, R5: 22, Resistor_SMD:R_0805_2012Metric, symbol Device:R_Small
Connections:
- net D+: now also R2.2; no longer U1.4 (D+)
- net D-: now also R5.2; no longer U1.3 (D-)
- new net: R5.1, U1.3 (D-)
- new net: R2.1, U1.4 (D+)
Changed lines of the file:
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@@
     (stroke (width 0) (type solid) (color 0 0 0 0))
   )
+  (wire (pts (xy 27.94 85.09) (xy 38.1 85.09))
+    (stroke (width 0) (type solid) (color 0 0 0 0))
+  )
+  (wire (pts (xy 29.21 91.44) (xy 33.02 91.44))
+    (stroke (width 0) (type solid) (color 0 0 0 0))
+  )
   (wire (pts (xy 29.21 233.68) (xy 29.21 241.3))
     (stroke (width 0) (type solid) (color 0 0 0 0))
@@
     (stroke (width 0) (type solid) (color 0 0 0 0))
   )
+  (wire (pts (xy 38.1 91.44) (xy 53.34 91.44))
+    (stroke (width 0) (type solid) (color 0 0 0 0))
+  )
   (wire (pts (xy 38.1 113.03) (xy 38.1 109.22))
     (stroke (width 0) (type solid) (color 0 0 0 0))
@@
     (stroke (width 0) (type solid) (color 0 0 0 0))
   )
+  (wire (pts (xy 43.18 85.09) (xy 57.15 85.09))
+    (stroke (width 0) (type solid) (color 0 0 0 0))
+  )
   (wire (pts (xy 45.72 62.23) (xy 45.72 64.77))
     (stroke (width 0) (type solid) (color 0 0 0 0))
@@
     (stroke (width 0) (type solid) (color 0 0 0 0))
   )
+  (wire (pts (xy 53.34 87.63) (xy 57.15 87.63))
+    (stroke (width 0) (type solid) (color 0 0 0 0))
+  )
+  (wire (pts (xy 53.34 91.44) (xy 53.34 87.63))
+    (stroke (width 0) (type solid) (color 0 0 0 0))
+  )
   (wire (pts (xy 54.61 259.08) (xy 54.61 254))
     (stroke (width 0) (type solid) (color 0 0 0 0))
@@
     (stroke (width 0) (type solid) (color 0 0 0 0))
   )
-  (global_label "D-" (shape input) (at 38.1 177.8 180) (fields_autoplaced)
+  (global_label "D+" (shape input) (at 27.94 85.09 180) (fields_autoplaced)
     (effects (font (size 1.27 1.27)) (justify right))
-    (property "Intersheet References" "${INTERSHEET_REFS}" (id 0) (at 0 -39.37 0)
+    (property "Intersheet References" "${INTERSHEET_REFS}" (id 0) (at -21.59 -41.91 0)
       (effects (font (size 1.27 1.27)) hide)
     )
   )
-  (global_label "D+" (shape input) (at 38.1 180.34 180) (fields_autoplaced)
+  (global_label "D-" (shape input) (at 29.21 91.44 180) (fields_autoplaced)
     (effects (font (size 1.27 1.27)) (justify right))
-    (property "Intersheet References" "${INTERSHEET_REFS}" (id 0) (at 0 -39.37 0)
+    (property "Intersheet References" "${INTERSHEET_REFS}" (id 0) (at -20.32 -38.1 0)
       (effects (font (size 1.27 1.27)) hide)
     )
   )
-  (global_label "D+" (shape input) (at 57.15 85.09 180) (fields_autoplaced)
+  (global_label "D-" (shape input) (at 38.1 177.8 180) (fields_autoplaced)
     (effects (font (size 1.27 1.27)) (justify right))
-    (property "Intersheet References" "${INTERSHEET_REFS}" (id 0) (at 7.62 -41.91 0)
+    (property "Intersheet References" "${INTERSHEET_REFS}" (id 0) (at 0 -39.37 0)
       (effects (font (size 1.27 1.27)) hide)
     )
   )
-  (global_label "D-" (shape input) (at 57.15 87.63 180) (fields_autoplaced)
+  (global_label "D+" (shape input) (at 38.1 180.34 180) (fields_autoplaced)
     (effects (font (size 1.27 1.27)) (justify right))
-    (property "Intersheet References" "${INTERSHEET_REFS}" (id 0) (at 7.62 -41.91 0)
+    (property "Intersheet References" "${INTERSHEET_REFS}" (id 0) (at 0 -39.37 0)
       (effects (font (size 1.27 1.27)) hide)
     )
@@
     (pin "1")
   )
+  (symbol (lib_id "Device:R_Small") (at 35.56 91.44 270) (unit 1)
+    (in_bom yes) (on_board yes)
+    (property "Reference" "R5" (id 0) (at 35.56 86.4616 90))
+    (property "Value" "22" (id 1) (at 35.56 88.773 90))
+    (property "Footprint" "Resistor_SMD:R_0805_2012Metric" (id 2) (at 35.56 91.44 0)
+      (effects (font (size 1.27 1.27)) hide)
+    )
+    (property "Datasheet" "~" (id 3) (at 35.56 91.44 0)
+      (effects (font (size 1.27 1.27)) hide)
+    )
+    (pin "1")
+    (pin "2")
+  )
+  (symbol (lib_id "Device:R_Small") (at 40.64 85.09 270) (unit 1)
+    (in_bom yes) (on_board yes)
+    (property "Reference" "R2" (id 0) (at 40.64 80.1116 90))
+    (property "Value" "22" (id 1) (at 40.64 82.423 90))
+    (property "Footprint" "Resistor_SMD:R_0805_2012Metric" (id 2) (at 40.64 85.09 0)
+      (effects (font (size 1.27 1.27)) hide)
+    )
+    (property "Datasheet" "~" (id 3) (at 40.64 85.09 0)
+      (effects (font (size 1.27 1.27)) hide)
+    )
+    (pin "1")
+    (pin "2")
+  )
   (symbol (lib_id "Device:R_Small") (at 57.15 39.37 180) (unit 1)
     (in_bom yes) (on_board yes)
@@
       (reference "R1") (unit 1) (value "330") (footprint "Resistor_SMD:R_0805_2012Metric")
     )
+    (path "/370e7d12-ac1a-44b1-8214-0db731e008f1"
+      (reference "R2") (unit 1) (value "22") (footprint "Resistor_SMD:R_0805_2012Metric")
+    )
     (path "/00000000-0000-0000-0000-000061280f1c"
       (reference "R3") (unit 1) (value "10k") (footprint "Resistor_SMD:R_0805_2012Metric")
@@
       (reference "R4") (unit 1) (value "10k") (footprint "Resistor_SMD:R_0805_2012Metric")
     )
+    (path "/86f546b5-aa43-4d36-9777-f9e527e27aec"
+      (reference "R5") (unit 1) (value "22") (footprint "Resistor_SMD:R_0805_2012Metric")
+    )
     (path "/00000000-0000-0000-0000-00006127121f"

Commit message: updates
Parts:
- renumbered R2 to R?, R5 to R?
Changed lines of the file:
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@@
   (symbol (lib_id "Device:R_Small") (at 35.56 91.44 270) (unit 1)
     (in_bom yes) (on_board yes)
-    (property "Reference" "R5" (id 0) (at 35.56 86.4616 90))
+    (property "Reference" "R?" (id 0) (at 35.56 86.4616 90))
     (property "Value" "22" (id 1) (at 35.56 88.773 90))
     (property "Footprint" "Resistor_SMD:R_0805_2012Metric" (id 2) (at 35.56 91.44 0)
@@
   (symbol (lib_id "Device:R_Small") (at 40.64 85.09 270) (unit 1)
     (in_bom yes) (on_board yes)
-    (property "Reference" "R2" (id 0) (at 40.64 80.1116 90))
+    (property "Reference" "R?" (id 0) (at 40.64 80.1116 90))
     (property "Value" "22" (id 1) (at 40.64 82.423 90))
     (property "Footprint" "Resistor_SMD:R_0805_2012Metric" (id 2) (at 40.64 85.09 0)
@@
       (reference "R1") (unit 1) (value "330") (footprint "Resistor_SMD:R_0805_2012Metric")
     )
-    (path "/370e7d12-ac1a-44b1-8214-0db731e008f1"
-      (reference "R2") (unit 1) (value "22") (footprint "Resistor_SMD:R_0805_2012Metric")
-    )
     (path "/00000000-0000-0000-0000-000061280f1c"
       (reference "R3") (unit 1) (value "10k") (footprint "Resistor_SMD:R_0805_2012Metric")
@@
       (reference "R4") (unit 1) (value "10k") (footprint "Resistor_SMD:R_0805_2012Metric")
     )
+    (path "/370e7d12-ac1a-44b1-8214-0db731e008f1"
+      (reference "R?") (unit 1) (value "22") (footprint "Resistor_SMD:R_0805_2012Metric")
+    )
     (path "/86f546b5-aa43-4d36-9777-f9e527e27aec"
-      (reference "R5") (unit 1) (value "22") (footprint "Resistor_SMD:R_0805_2012Metric")
+      (reference "R?") (unit 1) (value "22") (footprint "Resistor_SMD:R_0805_2012Metric")
     )
     (path "/00000000-0000-0000-0000-00006127121f"

Commit message: update
Parts:
- added U2: ATmega32U4-AU, Package_DFN_QFN:QFN-44-1EP_7x7mm_P0.5mm_EP5.2x5.2mm, symbol MCU_Microchip_ATmega:ATmega32U4-AU
- gave numbers to parts that had none: 2
Connections:
- net +5V: now also U2.14 (VCC), U2.2 (UVCC), U2.24 (AVCC), U2.34 (VCC), U2.44 (AVCC), U2.7 (VBUS)
- net BUZIN: now also U2.31 (PC6)
- net COL0: now also U2.41 (PF0)
- net COL1: now also U2.40 (PF1)
- net COL2: now also U2.38 (PF5)
- net COL3: now also U2.37 (PF6)
- net COL4: now also U2.36 (PF7)
- net COL5: now also U2.30 (PB6)
- net COL6: now also U2.29 (PB5)
- net COL7: now also U2.28 (PB4)
- net COL8: now also U2.26 (PD6)
- net COL9: now also U2.8 (PB0)
- net GND: now also U2.15 (GND), U2.23 (GND), U2.35 (GND), U2.43 (GND), U2.5 (UGND)
- net ROW0: now also U2.27 (PD7)
- net ROW1: now also U2.18 (PD0)
- net ROW10: now also U2.20 (PD2)
- net ROW2: now also U2.9 (PB1)
- net ROW3: now also U2.11 (PB3)
- net ROW4: now also U2.21 (PD3)
- net ROW5: now also U2.25 (PD4)
- net ROW6: now also U2.22 (PD5)
- net ROW7: now also U2.12 (PB7)
- net ROW8: now also U2.10 (PB2)
- net ROW9: now also U2.19 (PD1)
- net at U1.1 (PE6): now also U2.1 (PE6)
- net at R3.1, SW1.2, U1.13 (~{RESET}): now also U2.13 (~{RESET})
- net at C4.1, U1.16 (XTAL2), Y1.3: now also U2.16 (XTAL2)
- net at C3.1, U1.17 (XTAL1), Y1.1: now also U2.17 (XTAL1)
- net at R5.1, U1.3 (D-): now also U2.3 (D-)
- net at U1.32 (PC7): now also U2.32 (PC7)
- net at R4.2, U1.33 (~{HWB}/PE2): now also U2.33 (~{HWB}/PE2)
- net at R1.2, U1.39 (PF4): now also U2.39 (PF4)
- net at R2.1, U1.4 (D+): now also U2.4 (D+)
- net at U1.42 (AREF): now also U2.42 (AREF)
- net at C6.1, U1.6 (UCAP): now also U2.6 (UCAP)
Changed lines of the file:
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@@
   (junction (at 45.72 69.85) (diameter 1.016) (color 0 0 0 0))
   (junction (at 57.15 45.72) (diameter 1.016) (color 0 0 0 0))
+  (junction (at 57.15 59.69) (diameter 1.016) (color 0 0 0 0))
+  (junction (at 57.15 64.77) (diameter 1.016) (color 0 0 0 0))
+  (junction (at 57.15 69.85) (diameter 1.016) (color 0 0 0 0))
+  (junction (at 57.15 80.01) (diameter 1.016) (color 0 0 0 0))
+  (junction (at 57.15 85.09) (diameter 1.016) (color 0 0 0 0))
+  (junction (at 57.15 87.63) (diameter 1.016) (color 0 0 0 0))
+  (junction (at 57.15 92.71) (diameter 1.016) (color 0 0 0 0))
   (junction (at 64.77 233.68) (diameter 1.016) (color 0 0 0 0))
   (junction (at 64.77 241.3) (diameter 1.016) (color 0 0 0 0))
@@
   (junction (at 69.85 143.51) (diameter 1.016) (color 0 0 0 0))
   (junction (at 72.39 52.07) (diameter 1.016) (color 0 0 0 0))
+  (junction (at 72.39 143.51) (diameter 1.016) (color 0 0 0 0))
+  (junction (at 74.93 52.07) (diameter 1.016) (color 0 0 0 0))
+  (junction (at 87.63 113.03) (diameter 1.016) (color 0 0 0 0))
+  (junction (at 87.63 125.73) (diameter 1.016) (color 0 0 0 0))
   (junction (at 100.33 241.3) (diameter 1.016) (color 0 0 0 0))
   (junction (at 157.48 55.88) (diameter 1.016) (color 0 0 0 0))
@@
   (symbol (lib_id "Device:R_Small") (at 35.56 91.44 270) (unit 1)
     (in_bom yes) (on_board yes)
-    (property "Reference" "R?" (id 0) (at 35.56 86.4616 90))
+    (property "Reference" "R5" (id 0) (at 35.56 86.4616 90))
     (property "Value" "22" (id 1) (at 35.56 88.773 90))
     (property "Footprint" "Resistor_SMD:R_0805_2012Metric" (id 2) (at 35.56 91.44 0)
@@
   (symbol (lib_id "Device:R_Small") (at 40.64 85.09 270) (unit 1)
     (in_bom yes) (on_board yes)
-    (property "Reference" "R?" (id 0) (at 40.64 80.1116 90))
+    (property "Reference" "R2" (id 0) (at 40.64 80.1116 90))
     (property "Value" "22" (id 1) (at 40.64 82.423 90))
     (property "Footprint" "Resistor_SMD:R_0805_2012Metric" (id 2) (at 40.64 85.09 0)
@@
     (pin "9")
   )
+  (symbol (lib_id "MCU_Microchip_ATmega:ATmega32U4-AU") (at 72.39 97.79 0) (unit 1)
+    (in_bom yes) (on_board yes)
+    (property "Reference" "U2" (id 0) (at 72.39 145.7706 0))
+    (property "Value" "ATmega32U4-AU" (id 1) (at 72.39 148.082 0))
+    (property "Footprint" "Package_DFN_QFN:QFN-44-1EP_7x7mm_P0.5mm_EP5.2x5.2mm" (id 2) (at 72.39 97.79 0)
+      (effects (font (size 1.27 1.27) italic) hide)
+    )
+    (property "Datasheet" "http://ww1.microchip.com/downloads/en/DeviceDoc/Atmel-7766-8-bit-AVR-ATmega16U4-32U4_Datasheet.pdf" (id 3) (at 72.39 97.79 0)
+      (effects (font (size 1.27 1.27)) hide)
+    )
+    (pin "1")
+    (pin "10")
+    (pin "11")
+    (pin "12")
+    (pin "13")
+    (pin "14")
+    (pin "15")
+    (pin "16")
+    (pin "17")
+    (pin "18")
+    (pin "19")
+    (pin "2")
+    (pin "20")
+    (pin "21")
+    (pin "22")
+    (pin "23")
+    (pin "24")
+    (pin "25")
+    (pin "26")
+    (pin "27")
+    (pin "28")
+    (pin "29")
+    (pin "3")
+    (pin "30")
+    (pin "31")
+    (pin "32")
+    (pin "33")
+    (pin "34")
+    (pin "35")
+    (pin "36")
+    (pin "37")
+    (pin "38")
+    (pin "39")
+    (pin "4")
+    (pin "40")
+    (pin "41")
+    (pin "42")
+    (pin "43")
+    (pin "44")
+    (pin "5")
+    (pin "6")
+    (pin "7")
+    (pin "8")
+    (pin "9")
+  )
   (sheet_instances
     (path "/" (page "1"))
@@
       (reference "R1") (unit 1) (value "330") (footprint "Resistor_SMD:R_0805_2012Metric")
     )
+    (path "/370e7d12-ac1a-44b1-8214-0db731e008f1"
+      (reference "R2") (unit 1) (value "22") (footprint "Resistor_SMD:R_0805_2012Metric")
+    )
     (path "/00000000-0000-0000-0000-000061280f1c"
       (reference "R3") (unit 1) (value "10k") (footprint "Resistor_SMD:R_0805_2012Metric")
@@
       (reference "R4") (unit 1) (value "10k") (footprint "Resistor_SMD:R_0805_2012Metric")
     )
-    (path "/370e7d12-ac1a-44b1-8214-0db731e008f1"
-      (reference "R?") (unit 1) (value "22") (footprint "Resistor_SMD:R_0805_2012Metric")
-    )
     (path "/86f546b5-aa43-4d36-9777-f9e527e27aec"
-      (reference "R?") (unit 1) (value "22") (footprint "Resistor_SMD:R_0805_2012Metric")
+      (reference "R5") (unit 1) (value "22") (footprint "Resistor_SMD:R_0805_2012Metric")
     )
     (path "/00000000-0000-0000-0000-00006127121f"
@@
       (reference "U1") (unit 1) (value "ATmega32U4-AU") (footprint "Package_QFP:TQFP-44_10x10mm_P0.8mm")
     )
+    (path "/2ccdb65d-62ed-42d5-acea-df4cedf22149"
+      (reference "U2") (unit 1) (value "ATmega32U4-AU") (footprint "Package_DFN_QFN:QFN-44-1EP_7x7mm_P0.5mm_EP5.2x5.2mm")
+    )
     (path "/00000000-0000-0000-0000-0000612269b2"
