File: aek.kicad_sch (KiCad schematic)
At the start: 241 parts, among them J1 Conn_01x04_MountingPin, SW1 SW_Push, U1 ATmega32U4-MU, Y1 16MHz

Commit message: cleanup & onboard AST1109MLQ
Parts:
- added C11: 0.1uF, Capacitor_SMD:C_0805_2012Metric, symbol Device:C_Small
- added R6: 22, Resistor_SMD:R_0805_2012Metric, symbol Device:R_Small
- BUZ1: footprint Buzzer_Beeper:Buzzer_TDK_PS1240P02BT_D12.2mm_H6.5mm -> Buzzer_Beeper:Buzzer_Mallory_AST1109MLTRQ
Connections:
- net BUZIN: now also R6.1; no longer BUZ1.1
- net GND: now also C11.2
- new net: BUZ1.1, C11.1, R6.2
Other:
- moved on the sheet: BUZ1
Changed lines of the file:
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@@
   (junction (at 66.04 41.91) (diameter 1.016) (color 0 0 0 0))
   (junction (at 100.33 241.3) (diameter 1.016) (color 0 0 0 0))
+  (junction (at 114.3 186.69) (diameter 1.016) (color 0 0 0 0))
   (junction (at 157.48 55.88) (diameter 1.016) (color 0 0 0 0))
   (junction (at 157.48 74.93) (diameter 1.016) (color 0 0 0 0))
@@
     (stroke (width 0) (type solid) (color 0 0 0 0))
   )
-  (wire (pts (xy 19.05 222.25) (xy 19.05 226.06))
-    (stroke (width 0) (type solid) (color 0 0 0 0))
-  )
-  (wire (pts (xy 19.05 222.25) (xy 22.86 222.25))
-    (stroke (width 0) (type solid) (color 0 0 0 0))
-  )
   (wire (pts (xy 21.59 74.93) (xy 31.75 74.93))
     (stroke (width 0) (type solid) (color 0 0 0 0))
@@
     (stroke (width 0) (type solid) (color 0 0 0 0))
   )
-  (wire (pts (xy 27.94 222.25) (xy 33.02 222.25))
-    (stroke (width 0) (type solid) (color 0 0 0 0))
-  )
   (wire (pts (xy 29.21 233.68) (xy 29.21 241.3))
     (stroke (width 0) (type solid) (color 0 0 0 0))
@@
     (stroke (width 0) (type solid) (color 0 0 0 0))
   )
+  (wire (pts (xy 100.33 186.69) (xy 100.33 196.85))
+    (stroke (width 0) (type solid) (color 0 0 0 0))
+  )
+  (wire (pts (xy 100.33 186.69) (xy 105.41 186.69))
+    (stroke (width 0) (type solid) (color 0 0 0 0))
+  )
   (wire (pts (xy 100.33 233.68) (xy 100.33 241.3))
     (stroke (width 0) (type solid) (color 0 0 0 0))
@@
     (stroke (width 0) (type solid) (color 0 0 0 0))
   )
+  (wire (pts (xy 110.49 186.69) (xy 114.3 186.69))
+    (stroke (width 0) (type solid) (color 0 0 0 0))
+  )
+  (wire (pts (xy 114.3 186.69) (xy 114.3 189.23))
+    (stroke (width 0) (type solid) (color 0 0 0 0))
+  )
+  (wire (pts (xy 114.3 186.69) (xy 116.84 186.69))
+    (stroke (width 0) (type solid) (color 0 0 0 0))
+  )
+  (wire (pts (xy 114.3 194.31) (xy 114.3 196.85))
+    (stroke (width 0) (type solid) (color 0 0 0 0))
+  )
+  (wire (pts (xy 121.92 186.69) (xy 127 186.69))
+    (stroke (width 0) (type solid) (color 0 0 0 0))
+  )
   (wire (pts (xy 125.73 264.16) (xy 125.73 270.51))
     (stroke (width 0) (type solid) (color 0 0 0 0))
@@
     )
   )
-  (global_label "BUZIN" (shape input) (at 33.02 222.25 0) (fields_autoplaced)
-    (effects (font (size 1.27 1.27)) (justify left))
-    (property "Intersheet References" "${INTERSHEET_REFS}" (id 0) (at 41.0386 222.1706 0)
-      (effects (font (size 1.27 1.27)) (justify left) hide)
-    )
-  )
   (global_label "D-" (shape input) (at 45.72 177.8 0) (fields_autoplaced)
     (effects (font (size 1.27 1.27)) (justify left))
@@
     )
   )
+  (global_label "BUZIN" (shape input) (at 127 186.69 0) (fields_autoplaced)
+    (effects (font (size 1.27 1.27)) (justify left))
+    (property "Intersheet References" "${INTERSHEET_REFS}" (id 0) (at 135.0186 186.6106 0)
+      (effects (font (size 1.27 1.27)) (justify left) hide)
+    )
+  )
   (global_label "LEDDIN" (shape input) (at 133.35 254 0) (fields_autoplaced)
     (effects (font (size 1.27 1.27)) (justify left))
@@
     (pin "1")
   )
-  (symbol (lib_id "power:GND") (at 19.05 226.06 0) (unit 1)
-    (in_bom yes) (on_board yes)
-    (property "Reference" "#PWR0115" (id 0) (at 19.05 232.41 0)
-      (effects (font (size 1.27 1.27)) hide)
-    )
-    (property "Value" "GND" (id 1) (at 19.177 230.4542 0))
-    (property "Footprint" "" (id 2) (at 19.05 226.06 0)
-      (effects (font (size 1.27 1.27)) hide)
-    )
-    (property "Datasheet" "" (id 3) (at 19.05 226.06 0)
-      (effects (font (size 1.27 1.27)) hide)
-    )
-    (pin "1")
-  )
   (symbol (lib_id "power:GND") (at 24.13 64.77 0) (unit 1)
     (in_bom yes) (on_board yes)
@@
     (pin "1")
   )
+  (symbol (lib_id "power:GND") (at 100.33 196.85 0) (unit 1)
+    (in_bom yes) (on_board yes)
+    (property "Reference" "#PWR0115" (id 0) (at 100.33 203.2 0)
+      (effects (font (size 1.27 1.27)) hide)
+    )
+    (property "Value" "GND" (id 1) (at 100.457 201.2442 0))
+    (property "Footprint" "" (id 2) (at 100.33 196.85 0)
+      (effects (font (size 1.27 1.27)) hide)
+    )
+    (property "Datasheet" "" (id 3) (at 100.33 196.85 0)
+      (effects (font (size 1.27 1.27)) hide)
+    )
+    (pin "1")
+  )
   (symbol (lib_id "power:GND") (at 110.49 241.3 90) (unit 1)
     (in_bom yes) (on_board yes)
@@
     (pin "1")
   )
-  (symbol (lib_id "power:GND") (at 125.73 270.51 0) (unit 1)
+  (symbol (lib_id "power:GND") (at 114.3 196.85 0) (unit 1)
     (in_bom yes) (on_board yes)
-    (property "Reference" "#PWR0120" (id 0) (at 125.73 276.86 0)
+    (property "Reference" "#PWR0123" (id 0) (at 114.3 203.2 0)
       (effects (font (size 1.27 1.27)) hide)
     )
-    (property "Value" "GND" (id 1) (at 125.857 274.9042 0))
-    (property "Footprint" "" (id 2) (at 125.73 270.51 0)
+    (property "Value" "GND" (id 1) (at 114.427 201.2442 0))
+    (property "Footprint" "" (id 2) (at 114.3 196.85 0)
       (effects (font (size 1.27 1.27)) hide)
     )
-    (property "Datasheet" "" (id 3) (at 125.73 270.51 0)
+    (property "Datasheet" "" (id 3) (at 114.3 196.85 0)
       (effects (font (size 1.27 1.27)) hide)
     )
     (pin "1")
   )
-  (symbol (lib_id "Device:R_Small") (at 25.4 222.25 270) (unit 1)
+  (symbol (lib_id "power:GND") (at 125.73 270.51 0) (unit 1)
     (in_bom yes) (on_board yes)
-    (property "Reference" "BUZ1" (id 0) (at 25.4 217.2716 90))
-    (property "Value" "Buzzer" (id 1) (at 25.4 219.583 90))
-    (property "Footprint" "Buzzer_Beeper:Buzzer_TDK_PS1240P02BT_D12.2mm_H6.5mm" (id 2) (at 25.4 222.25 0)
+    (property "Reference" "#PWR0120" (id 0) (at 125.73 276.86 0)
       (effects (font (size 1.27 1.27)) hide)
     )
-    (property "Datasheet" "~" (id 3) (at 25.4 222.25 0)
+    (property "Value" "GND" (id 1) (at 125.857 274.9042 0))
+    (property "Footprint" "" (id 2) (at 125.73 270.51 0)
+      (effects (font (size 1.27 1.27)) hide)
+    )
+    (property "Datasheet" "" (id 3) (at 125.73 270.51 0)
       (effects (font (size 1.27 1.27)) hide)
     )
     (pin "1")
-    (pin "2")
   )
   (symbol (lib_id "Device:R_Small") (at 29.21 81.28 270) (unit 1)
@@
     (pin "2")
   )
+  (symbol (lib_id "Device:R_Small") (at 107.95 186.69 270) (unit 1)
+    (in_bom yes) (on_board yes)
+    (property "Reference" "BUZ1" (id 0) (at 107.95 181.7116 90))
+    (property "Value" "Buzzer" (id 1) (at 107.95 184.023 90))
+    (property "Footprint" "Buzzer_Beeper:Buzzer_Mallory_AST1109MLTRQ" (id 2) (at 107.95 186.69 0)
+      (effects (font (size 1.27 1.27)) hide)
+    )
+    (property "Datasheet" "~" (id 3) (at 107.95 186.69 0)
+      (effects (font (size 1.27 1.27)) hide)
+    )
+    (pin "1")
+    (pin "2")
+  )
+  (symbol (lib_id "Device:R_Small") (at 119.38 186.69 270) (unit 1)
+    (in_bom yes) (on_board yes)
+    (property "Reference" "R6" (id 0) (at 119.38 181.7116 90))
+    (property "Value" "22" (id 1) (at 119.38 184.023 90))
+    (property "Footprint" "Resistor_SMD:R_0805_2012Metric" (id 2) (at 119.38 186.69 0)
+      (effects (font (size 1.27 1.27)) hide)
+    )
+    (property "Datasheet" "~" (id 3) (at 119.38 186.69 0)
+      (effects (font (size 1.27 1.27)) hide)
+    )
+    (pin "1")
+    (pin "2")
+  )
   (symbol (lib_id "Device:D_Small") (at 157.48 53.34 90) (unit 1)
     (in_bom yes) (on_board yes)
@@
     (pin "2")
   )
+  (symbol (lib_id "Device:C_Small") (at 114.3 191.77 0) (mirror y) (unit 1)
+    (in_bom yes) (on_board yes)
+    (property "Reference" "C11" (id 0) (at 111.9632 190.6016 0)
+      (effects (font (size 1.27 1.27)) (justify left))
+    )
+    (property "Value" "0.1uF" (id 1) (at 111.9632 192.913 0)
+      (effects (font (size 1.27 1.27)) (justify left))
+    )
+    (property "Footprint" "Capacitor_SMD:C_0805_2012Metric" (id 2) (at 114.3 191.77 0)
+      (effects (font (size 1.27 1.27)) hide)
+    )
+    (property "Datasheet" "~" (id 3) (at 114.3 191.77 0)
+      (effects (font (size 1.27 1.27)) hide)
+    )
+    (pin "1")
+    (pin "2")
+  )
   (symbol (lib_id "Mechanical:MountingHole_Pad") (at 17.78 201.93 0) (unit 1)
     (in_bom yes) (on_board yes)
@@
       (reference "#PWR0122") (unit 1) (value "GND") (footprint "")
     )
+    (path "/f1a3a060-6bd3-44d7-bff1-afaf1ec0bb82"
+      (reference "#PWR0123") (unit 1) (value "GND") (footprint "")
+    )
     (path "/5e7696e2-7dd3-4741-abb9-0ce915833473"
-      (reference "BUZ1") (unit 1) (value "Buzzer") (footprint "Buzzer_Beeper:Buzzer_TDK_PS1240P02BT_D12.2mm_H6.5mm")
+      (reference "BUZ1") (unit 1) (value "Buzzer") (footprint "Buzzer_Beeper:Buzzer_Mallory_AST1109MLTRQ")
     )
     (path "/00000000-0000-0000-0000-00006120a5a3"
@@
       (reference "C10") (unit 1) (value "0.1uF") (footprint "Capacitor_SMD:C_0805_2012Metric")
     )
+    (path "/a54f80d2-1af3-49fe-91f4-944ea459bf74"
+      (reference "C11") (unit 1) (value "0.1uF") (footprint "Capacitor_SMD:C_0805_2012Metric")
+    )
     (path "/00000000-0000-0000-0000-000061242afa"
       (reference "D1") (unit 1) (value "D_Small") (footprint "Diode_SMD:D_SOD-123")
@@
       (reference "R5") (unit 1) (value "22") (footprint "Resistor_SMD:R_0805_2012Metric")
     )
+    (path "/687cebef-2528-423d-a3e0-77332de3f6f2"
+      (reference "R6") (unit 1) (value "22") (footprint "Resistor_SMD:R_0805_2012Metric")
+    )
     (path "/00000000-0000-0000-0000-00006127121f"

Commit message: updates
Parts:
- added LED4, LED5, LED6: WS2812B, LED_SMD:LED_WS2812B_PLCC4_5.0x5.0mm_P3.2mm, symbol ws2812b:WS2812B
- LED1, LED2, LED3: footprint LED_SMD:LED_WS2812B_PLCC4_5.0x5.0mm_P3.2mm -> LED_THT:LED_D5.0mm-4_RGB
Connections:
- net +5V: now also LED4.1 (VCC), LED5.1 (VCC), LED6.1 (VCC)
- net GND: now also LED4.3 (GND), LED5.3 (GND), LED6.3 (GND)
- net LEDDIN: now also LED6.4 (DIN)
- net at LED1.2 (DOUT): now also LED4.2 (DOUT)
- net at LED1.4 (DIN), LED2.2 (DOUT): now also LED4.4 (DIN), LED5.2 (DOUT)
- net at LED2.4 (DIN), LED3.2 (DOUT): now also LED5.4 (DIN), LED6.2 (DOUT)
Changed lines of the file:
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@@
   (junction (at 27.94 64.77) (diameter 1.016) (color 0 0 0 0))
   (junction (at 29.21 241.3) (diameter 1.016) (color 0 0 0 0))
+  (junction (at 29.21 254) (diameter 1.016) (color 0 0 0 0))
+  (junction (at 29.21 264.16) (diameter 1.016) (color 0 0 0 0))
   (junction (at 31.75 102.87) (diameter 1.016) (color 0 0 0 0))
   (junction (at 31.75 107.95) (diameter 1.016) (color 0 0 0 0))
@@
   (junction (at 50.8 35.56) (diameter 1.016) (color 0 0 0 0))
   (junction (at 53.34 170.18) (diameter 1.016) (color 0 0 0 0))
+  (junction (at 54.61 254) (diameter 1.016) (color 0 0 0 0))
+  (junction (at 54.61 264.16) (diameter 1.016) (color 0 0 0 0))
   (junction (at 63.5 41.91) (diameter 1.016) (color 0 0 0 0))
   (junction (at 63.5 133.35) (diameter 1.016) (color 0 0 0 0))
   (junction (at 64.77 233.68) (diameter 1.016) (color 0 0 0 0))
   (junction (at 64.77 241.3) (diameter 1.016) (color 0 0 0 0))
+  (junction (at 64.77 254) (diameter 1.016) (color 0 0 0 0))
+  (junction (at 64.77 264.16) (diameter 1.016) (color 0 0 0 0))
   (junction (at 66.04 41.91) (diameter 1.016) (color 0 0 0 0))
+  (junction (at 90.17 254) (diameter 1.016) (color 0 0 0 0))
+  (junction (at 90.17 264.16) (diameter 1.016) (color 0 0 0 0))
   (junction (at 100.33 241.3) (diameter 1.016) (color 0 0 0 0))
+  (junction (at 100.33 254) (diameter 1.016) (color 0 0 0 0))
+  (junction (at 100.33 264.16) (diameter 1.016) (color 0 0 0 0))
   (junction (at 114.3 186.69) (diameter 1.016) (color 0 0 0 0))
+  (junction (at 125.73 254) (diameter 1.016) (color 0 0 0 0))
+  (junction (at 125.73 264.16) (diameter 1.016) (color 0 0 0 0))
   (junction (at 157.48 55.88) (diameter 1.016) (color 0 0 0 0))
   (junction (at 157.48 74.93) (diameter 1.016) (color 0 0 0 0))
@@
       (effects (font (size 1.524 1.524)))
     )
+    (property "Footprint" "LED_THT:LED_D5.0mm-4_RGB" (id 2) (at 41.91 249.4026 0)
+      (effects (font (size 1.524 1.524)) hide)
+    )
+    (property "Datasheet" "" (id 3) (at 40.64 259.08 90)
+      (effects (font (size 1.524 1.524)))
+    )
+    (pin "1")
+    (pin "2")
+    (pin "3")
+    (pin "4")
+  )
+  (symbol (lib_id "ws2812b:WS2812B") (at 41.91 259.08 0) (unit 1)
+    (in_bom yes) (on_board yes)
+    (property "Reference" "LED4" (id 0) (at 41.91 246.7102 0)
+      (effects (font (size 1.524 1.524)))
+    )
+    (property "Value" "WS2812B" (id 1) (at 41.91 249.4026 0)
+      (effects (font (size 1.524 1.524)))
+    )
     (property "Footprint" "LED_SMD:LED_WS2812B_PLCC4_5.0x5.0mm_P3.2mm" (id 2) (at 41.91 249.4026 0)
       (effects (font (size 1.524 1.524)) hide)
@@
       (effects (font (size 1.524 1.524)))
     )
+    (property "Footprint" "LED_THT:LED_D5.0mm-4_RGB" (id 2) (at 77.47 249.4026 0)
+      (effects (font (size 1.524 1.524)) hide)
+    )
+    (property "Datasheet" "" (id 3) (at 76.2 259.08 90)
+      (effects (font (size 1.524 1.524)))
+    )
+    (pin "1")
+    (pin "2")
+    (pin "3")
+    (pin "4")
+  )
+  (symbol (lib_id "ws2812b:WS2812B") (at 77.47 259.08 0) (unit 1)
+    (in_bom yes) (on_board yes)
+    (property "Reference" "LED5" (id 0) (at 77.47 246.7102 0)
+      (effects (font (size 1.524 1.524)))
+    )
+    (property "Value" "WS2812B" (id 1) (at 77.47 249.4026 0)
+      (effects (font (size 1.524 1.524)))
+    )
     (property "Footprint" "LED_SMD:LED_WS2812B_PLCC4_5.0x5.0mm_P3.2mm" (id 2) (at 77.47 249.4026 0)
       (effects (font (size 1.524 1.524)) hide)
@@
       (effects (font (size 1.524 1.524)))
     )
+    (property "Footprint" "LED_THT:LED_D5.0mm-4_RGB" (id 2) (at 113.03 249.4026 0)
+      (effects (font (size 1.524 1.524)) hide)
+    )
+    (property "Datasheet" "" (id 3) (at 111.76 259.08 90)
+      (effects (font (size 1.524 1.524)))
+    )
+    (pin "1")
+    (pin "2")
+    (pin "3")
+    (pin "4")
+  )
+  (symbol (lib_id "ws2812b:WS2812B") (at 113.03 259.08 0) (unit 1)
+    (in_bom yes) (on_board yes)
+    (property "Reference" "LED6" (id 0) (at 113.03 246.7102 0)
+      (effects (font (size 1.524 1.524)))
+    )
+    (property "Value" "WS2812B" (id 1) (at 113.03 249.4026 0)
+      (effects (font (size 1.524 1.524)))
+    )
     (property "Footprint" "LED_SMD:LED_WS2812B_PLCC4_5.0x5.0mm_P3.2mm" (id 2) (at 113.03 249.4026 0)
       (effects (font (size 1.524 1.524)) hide)
@@
     )
     (path "/00000000-0000-0000-0000-0000612394e1"
-      (reference "LED1") (unit 1) (value "WS2812B") (footprint "LED_SMD:LED_WS2812B_PLCC4_5.0x5.0mm_P3.2mm")
+      (reference "LED1") (unit 1) (value "WS2812B") (footprint "LED_THT:LED_D5.0mm-4_RGB")
     )
     (path "/00000000-0000-0000-0000-00006197b9d3"
-      (reference "LED2") (unit 1) (value "WS2812B") (footprint "LED_SMD:LED_WS2812B_PLCC4_5.0x5.0mm_P3.2mm")
+      (reference "LED2") (unit 1) (value "WS2812B") (footprint "LED_THT:LED_D5.0mm-4_RGB")
     )
     (path "/00000000-0000-0000-0000-00006197d290"
-      (reference "LED3") (unit 1) (value "WS2812B") (footprint "LED_SMD:LED_WS2812B_PLCC4_5.0x5.0mm_P3.2mm")
+      (reference "LED3") (unit 1) (value "WS2812B") (footprint "LED_THT:LED_D5.0mm-4_RGB")
+    )
+    (path "/28fbf76e-ce81-42d3-8fb7-a1863f0e3ee4"
+      (reference "LED4") (unit 1) (value "WS2812B") (footprint "LED_SMD:LED_WS2812B_PLCC4_5.0x5.0mm_P3.2mm")
+    )
+    (path "/79e95da9-b05b-48d5-8a04-48d4b7b6061a"
+      (reference "LED5") (unit 1) (value "WS2812B") (footprint "LED_SMD:LED_WS2812B_PLCC4_5.0x5.0mm_P3.2mm")
+    )
+    (path "/6e9bf1b0-f56c-41b3-a430-6f5502d4acea"
+      (reference "LED6") (unit 1) (value "WS2812B") (footprint "LED_SMD:LED_WS2812B_PLCC4_5.0x5.0mm_P3.2mm")
     )
     (path "/00000000-0000-0000-0000-00006130a8dc"

Commit message: update
Parts:
- removed LED4, LED5, LED6: WS2812B, LED_SMD:LED_WS2812B_PLCC4_5.0x5.0mm_P3.2mm, symbol ws2812b:WS2812B
- LED1, LED2, LED3: footprint LED_THT:LED_D5.0mm-4_RGB -> WS2812B:WS2812BDual
Changed lines of the file:
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@@
   (junction (at 27.94 64.77) (diameter 1.016) (color 0 0 0 0))
   (junction (at 29.21 241.3) (diameter 1.016) (color 0 0 0 0))
-  (junction (at 29.21 254) (diameter 1.016) (color 0 0 0 0))
-  (junction (at 29.21 264.16) (diameter 1.016) (color 0 0 0 0))
   (junction (at 31.75 102.87) (diameter 1.016) (color 0 0 0 0))
   (junction (at 31.75 107.95) (diameter 1.016) (color 0 0 0 0))
@@
   (junction (at 50.8 35.56) (diameter 1.016) (color 0 0 0 0))
   (junction (at 53.34 170.18) (diameter 1.016) (color 0 0 0 0))
-  (junction (at 54.61 254) (diameter 1.016) (color 0 0 0 0))
-  (junction (at 54.61 264.16) (diameter 1.016) (color 0 0 0 0))
   (junction (at 63.5 41.91) (diameter 1.016) (color 0 0 0 0))
   (junction (at 63.5 133.35) (diameter 1.016) (color 0 0 0 0))
   (junction (at 64.77 233.68) (diameter 1.016) (color 0 0 0 0))
   (junction (at 64.77 241.3) (diameter 1.016) (color 0 0 0 0))
-  (junction (at 64.77 254) (diameter 1.016) (color 0 0 0 0))
-  (junction (at 64.77 264.16) (diameter 1.016) (color 0 0 0 0))
   (junction (at 66.04 41.91) (diameter 1.016) (color 0 0 0 0))
-  (junction (at 90.17 254) (diameter 1.016) (color 0 0 0 0))
-  (junction (at 90.17 264.16) (diameter 1.016) (color 0 0 0 0))
   (junction (at 100.33 241.3) (diameter 1.016) (color 0 0 0 0))
-  (junction (at 100.33 254) (diameter 1.016) (color 0 0 0 0))
-  (junction (at 100.33 264.16) (diameter 1.016) (color 0 0 0 0))
   (junction (at 114.3 186.69) (diameter 1.016) (color 0 0 0 0))
-  (junction (at 125.73 254) (diameter 1.016) (color 0 0 0 0))
-  (junction (at 125.73 264.16) (diameter 1.016) (color 0 0 0 0))
   (junction (at 157.48 55.88) (diameter 1.016) (color 0 0 0 0))
   (junction (at 157.48 74.93) (diameter 1.016) (color 0 0 0 0))
@@
       (effects (font (size 1.524 1.524)))
     )
-    (property "Footprint" "LED_THT:LED_D5.0mm-4_RGB" (id 2) (at 41.91 249.4026 0)
-      (effects (font (size 1.524 1.524)) hide)
-    )
-    (property "Datasheet" "" (id 3) (at 40.64 259.08 90)
-      (effects (font (size 1.524 1.524)))
-    )
-    (pin "1")
-    (pin "2")
-    (pin "3")
-    (pin "4")
-  )
-  (symbol (lib_id "ws2812b:WS2812B") (at 41.91 259.08 0) (unit 1)
-    (in_bom yes) (on_board yes)
-    (property "Reference" "LED4" (id 0) (at 41.91 246.7102 0)
-      (effects (font (size 1.524 1.524)))
-    )
-    (property "Value" "WS2812B" (id 1) (at 41.91 249.4026 0)
-      (effects (font (size 1.524 1.524)))
-    )
-    (property "Footprint" "LED_SMD:LED_WS2812B_PLCC4_5.0x5.0mm_P3.2mm" (id 2) (at 41.91 249.4026 0)
+    (property "Footprint" "WS2812B:WS2812BDual" (id 2) (at 41.91 249.4026 0)
       (effects (font (size 1.524 1.524)) hide)
     )
@@
       (effects (font (size 1.524 1.524)))
     )
-    (property "Footprint" "LED_THT:LED_D5.0mm-4_RGB" (id 2) (at 77.47 249.4026 0)
-      (effects (font (size 1.524 1.524)) hide)
-    )
-    (property "Datasheet" "" (id 3) (at 76.2 259.08 90)
-      (effects (font (size 1.524 1.524)))
-    )
-    (pin "1")
-    (pin "2")
-    (pin "3")
-    (pin "4")
-  )
-  (symbol (lib_id "ws2812b:WS2812B") (at 77.47 259.08 0) (unit 1)
-    (in_bom yes) (on_board yes)
-    (property "Reference" "LED5" (id 0) (at 77.47 246.7102 0)
-      (effects (font (size 1.524 1.524)))
-    )
-    (property "Value" "WS2812B" (id 1) (at 77.47 249.4026 0)
-      (effects (font (size 1.524 1.524)))
-    )
-    (property "Footprint" "LED_SMD:LED_WS2812B_PLCC4_5.0x5.0mm_P3.2mm" (id 2) (at 77.47 249.4026 0)
+    (property "Footprint" "WS2812B:WS2812BDual" (id 2) (at 77.47 249.4026 0)
       (effects (font (size 1.524 1.524)) hide)
     )
@@
       (effects (font (size 1.524 1.524)))
     )
-    (property "Footprint" "LED_THT:LED_D5.0mm-4_RGB" (id 2) (at 113.03 249.4026 0)
-      (effects (font (size 1.524 1.524)) hide)
-    )
-    (property "Datasheet" "" (id 3) (at 111.76 259.08 90)
-      (effects (font (size 1.524 1.524)))
-    )
-    (pin "1")
-    (pin "2")
-    (pin "3")
-    (pin "4")
-  )
-  (symbol (lib_id "ws2812b:WS2812B") (at 113.03 259.08 0) (unit 1)
-    (in_bom yes) (on_board yes)
-    (property "Reference" "LED6" (id 0) (at 113.03 246.7102 0)
-      (effects (font (size 1.524 1.524)))
-    )
-    (property "Value" "WS2812B" (id 1) (at 113.03 249.4026 0)
-      (effects (font (size 1.524 1.524)))
-    )
-    (property "Footprint" "LED_SMD:LED_WS2812B_PLCC4_5.0x5.0mm_P3.2mm" (id 2) (at 113.03 249.4026 0)
+    (property "Footprint" "WS2812B:WS2812BDual" (id 2) (at 113.03 249.4026 0)
       (effects (font (size 1.524 1.524)) hide)
     )
@@
     )
     (path "/00000000-0000-0000-0000-0000612394e1"
-      (reference "LED1") (unit 1) (value "WS2812B") (footprint "LED_THT:LED_D5.0mm-4_RGB")
+      (reference "LED1") (unit 1) (value "WS2812B") (footprint "WS2812B:WS2812BDual")
     )
     (path "/00000000-0000-0000-0000-00006197b9d3"
-      (reference "LED2") (unit 1) (value "WS2812B") (footprint "LED_THT:LED_D5.0mm-4_RGB")
+      (reference "LED2") (unit 1) (value "WS2812B") (footprint "WS2812B:WS2812BDual")
     )
     (path "/00000000-0000-0000-0000-00006197d290"
-      (reference "LED3") (unit 1) (value "WS2812B") (footprint "LED_THT:LED_D5.0mm-4_RGB")
-    )
-    (path "/28fbf76e-ce81-42d3-8fb7-a1863f0e3ee4"
-      (reference "LED4") (unit 1) (value "WS2812B") (footprint "LED_SMD:LED_WS2812B_PLCC4_5.0x5.0mm_P3.2mm")
-    )
-    (path "/79e95da9-b05b-48d5-8a04-48d4b7b6061a"
-      (reference "LED5") (unit 1) (value "WS2812B") (footprint "LED_SMD:LED_WS2812B_PLCC4_5.0x5.0mm_P3.2mm")
-    )
-    (path "/6e9bf1b0-f56c-41b3-a430-6f5502d4acea"
-      (reference "LED6") (unit 1) (value "WS2812B") (footprint "LED_SMD:LED_WS2812B_PLCC4_5.0x5.0mm_P3.2mm")
+      (reference "LED3") (unit 1) (value "WS2812B") (footprint "WS2812B:WS2812BDual")
     )
     (path "/00000000-0000-0000-0000-00006130a8dc"
